Commit message: update

File: nero/urdf/nero_description.urdf (robot description, URDF)
Before this commit: robot nero_description, 10 links, 9 joints
Joints:
- joint joint1: limit lower=-2.7 upper=2.7 effort=0 velocity=0 -> lower=-2.7 upper=2.7 effort=100 velocity=10
- joint joint2: limit lower=-1.74 upper=1.74 effort=0 velocity=0 -> lower=-1.74 upper=1.74 effort=100 velocity=10
- joint joint3: limit lower=-2.75 upper=2.75 effort=0 velocity=0 -> lower=-2.75 upper=2.75 effort=100 velocity=10
- joint joint4: limit lower=-1.01 upper=2.14 effort=0 velocity=0 -> lower=-1.01 upper=2.14 effort=100 velocity=10
- joint joint5: limit lower=-2.75 upper=2.75 effort=0 velocity=0 -> lower=-2.75 upper=2.75 effort=100 velocity=10
- joint joint6: limit lower=-0.73 upper=0.95 effort=0 velocity=0 -> lower=-0.73 upper=0.95 effort=100 velocity=10
- joint joint7: limit lower=-1.57 upper=1.57 effort=0 velocity=0 -> lower=-1.57 upper=1.57 effort=100 velocity=10

File: nero/urdf/nero_description_stand_v2.urdf (robot description, URDF)
Before this commit: robot nero_description, 10 links, 9 joints
Joints:
- joint joint1: limit lower=-2.7 upper=2.7 effort=0 velocity=0 -> lower=-2.7 upper=2.7 effort=100 velocity=10
- joint joint2: limit lower=-1.74 upper=1.74 effort=0 velocity=0 -> lower=-1.74 upper=1.74 effort=100 velocity=10
- joint joint3: limit lower=-2.75 upper=2.75 effort=0 velocity=0 -> lower=-2.75 upper=2.75 effort=100 velocity=10
- joint joint4: limit lower=-1.01 upper=2.14 effort=0 velocity=0 -> lower=-1.01 upper=2.14 effort=100 velocity=10
- joint joint5: limit lower=-2.75 upper=2.75 effort=0 velocity=0 -> lower=-2.75 upper=2.75 effort=100 velocity=10
- joint joint6: limit lower=-0.73 upper=0.95 effort=0 velocity=0 -> lower=-0.73 upper=0.95 effort=100 velocity=10
- joint joint7: limit lower=-1.57 upper=1.57 effort=0 velocity=0 -> lower=-1.57 upper=1.57 effort=100 velocity=10

File: nero/urdf/nero_with_hand_flange_description.urdf (robot description, URDF)
Before this commit: robot nero_description, 10 links, 9 joints
Joints:
- joint joint1: limit lower=-2.7 upper=2.7 effort=0 velocity=0 -> lower=-2.7 upper=2.7 effort=100 velocity=10
- joint joint2: limit lower=-1.74 upper=1.74 effort=0 velocity=0 -> lower=-1.74 upper=1.74 effort=100 velocity=10
- joint joint3: limit lower=-2.75 upper=2.75 effort=0 velocity=0 -> lower=-2.75 upper=2.75 effort=100 velocity=10
- joint joint4: limit lower=-1.01 upper=2.14 effort=0 velocity=0 -> lower=-1.01 upper=2.14 effort=100 velocity=10
- joint joint5: limit lower=-2.75 upper=2.75 effort=0 velocity=0 -> lower=-2.75 upper=2.75 effort=100 velocity=10
- joint joint6: limit lower=-0.73 upper=0.95 effort=0 velocity=0 -> lower=-0.73 upper=0.95 effort=100 velocity=10
- joint joint7: limit lower=-1.57 upper=1.57 effort=0 velocity=0 -> lower=-1.57 upper=1.57 effort=100 velocity=10

File: piper_h/urdf/piper_h_description_dark.urdf (robot description, URDF)
Before this commit: robot piper_h_description, 7 links, 6 joints
Joints:
- joint joint1: limit lower=0 upper=0 effort=0 velocity=0 -> lower=0 upper=0 effort=100 velocity=10
- joint joint2: limit lower=0 upper=0 effort=0 velocity=0 -> lower=0 upper=0 effort=100 velocity=10
- joint joint3: limit lower=0 upper=0 effort=0 velocity=0 -> lower=0 upper=0 effort=100 velocity=10
- joint joint4: limit lower=0 upper=0 effort=0 velocity=0 -> lower=0 upper=0 effort=100 velocity=10
- joint joint5: limit lower=0 upper=0 effort=0 velocity=0 -> lower=0 upper=0 effort=100 velocity=10
- joint joint6: limit lower=0 upper=0 effort=0 velocity=0 -> lower=0 upper=0 effort=100 velocity=10
