Commit message: fix(urdf): 修正 Piper/Nero 末端连杆质量与惯量
- 将 Piper、Piper H、Piper L、Piper X 的 link6 质量更新为 0.00613114124 kg，并修正惯性张量
- 将 Nero 的 link7 质量由 0.000001 kg 调整为 0.001 kg

---

fix(urdf): correct Piper/Nero end-link mass and inertia

- Update link6 mass to 0.00613114124 kg and correct its inertia tensor for Piper, Piper H, Piper L and Piper X
- Change Nero link7 mass from 0.000001 kg to 0.001 kg

File: nero/urdf/nero_description.urdf (robot description, URDF)
Before this commit: robot nero, 9 links, 8 joints
Links:
- link link7: mass 0.000001 -> 0.001

File: piper/urdf/piper_description.urdf (robot description, URDF)
Before this commit: robot piper, 8 links, 7 joints
Links:
- link link6: mass 0.007 -> 0.00613114124

File: piper_h/urdf/piper_h_description.urdf (robot description, URDF)
Before this commit: robot piper_h, 8 links, 7 joints
Links:
- link link6: mass 0.007 -> 0.00613114124

File: piper_l/urdf/piper_l_description.urdf (robot description, URDF)
Before this commit: robot piper_l, 8 links, 7 joints
Links:
- link link6: mass 0.007 -> 0.00613114124

File: piper_x/urdf/piper_x_description.urdf (robot description, URDF)
Before this commit: robot piper_x, 8 links, 7 joints
Links:
- link link6: mass 0.007 -> 0.00613114124

Commit message: fix(urdf): 同步 Piper/Nero 末端连杆质量与惯量
- 同步 main 提交 9f45f05 的 link6/link7 质量与惯量修正
- 更新基础模型及夹爪、Revo2 和法兰组合的 22 个 URDF
- 保留当前分支的网格路径和目录结构

---

fix(urdf): sync Piper/Nero end-link mass and inertia

- Sync the link6/link7 mass and inertia corrections from main commit 9f45f05
- Update 22 URDF files covering base models, grippers, Revo2 hands and flange combinations
- Preserve branch-specific mesh paths and directory structure

File: nero/urdf/nero_description.urdf (robot description, URDF)
Before this commit: robot nero, 9 links, 8 joints
Links:
- link link7: mass 0.000001 -> 0.001

File: nero/urdf/nero_with_gripper_description.urdf (robot description, URDF)
Before this commit: robot nero, 14 links, 13 joints
Links:
- link link7: mass 0.000001 -> 0.001

File: nero/urdf/nero_with_gripper_flange_description.urdf (robot description, URDF)
Before this commit: robot nero, 10 links, 9 joints
Links:
- link link7: mass 0.000001 -> 0.001

File: nero/urdf/nero_with_left_revo2_description.urdf (robot description, URDF)
Before this commit: robot nero, 32 links, 31 joints
Links:
- link link7: mass 0.000001 -> 0.001

File: nero/urdf/nero_with_revo2_flange_description.urdf (robot description, URDF)
Before this commit: robot nero, 10 links, 9 joints
Links:
- link link7: mass 0.000001 -> 0.001

File: nero/urdf/nero_with_right_revo2_description.urdf (robot description, URDF)
Before this commit: robot nero, 32 links, 31 joints
Links:
- link link7: mass 0.000001 -> 0.001

File: piper/urdf/piper_description.urdf (robot description, URDF)
Before this commit: robot piper, 8 links, 7 joints
Links:
- link link6: mass 0.007 -> 0.00613114124

File: piper/urdf/piper_with_gripper_description.urdf (robot description, URDF)
Before this commit: robot piper, 13 links, 12 joints
Links:
- link link6: mass 0.007 -> 0.00613114124

File: piper/urdf/piper_with_left_revo2_description.urdf (robot description, URDF)
Before this commit: robot piper, 31 links, 30 joints
Links:
- link link6: mass 0.007 -> 0.00613114124

File: piper/urdf/piper_with_right_revo2_description.urdf (robot description, URDF)
Before this commit: robot piper, 31 links, 30 joints
Links:
- link link6: mass 0.007 -> 0.00613114124

File: piper_h/urdf/piper_h_description.urdf (robot description, URDF)
Before this commit: robot piper_h, 8 links, 7 joints
Links:
- link link6: mass 0.007 -> 0.00613114124

File: piper_h/urdf/piper_h_with_gripper_description.urdf (robot description, URDF)
Before this commit: robot piper_h, 13 links, 12 joints
Links:
- link link6: mass 0.007 -> 0.00613114124

File: piper_h/urdf/piper_h_with_left_revo2_description.urdf (robot description, URDF)
Before this commit: robot piper_h, 31 links, 30 joints
Links:
- link link6: mass 0.007 -> 0.00613114124

File: piper_h/urdf/piper_h_with_right_revo2_description.urdf (robot description, URDF)
Before this commit: robot piper_h, 31 links, 30 joints
Links:
- link link6: mass 0.007 -> 0.00613114124

File: piper_l/urdf/piper_l_description.urdf (robot description, URDF)
Before this commit: robot piper_l, 8 links, 7 joints
Links:
- link link6: mass 0.007 -> 0.00613114124

File: piper_l/urdf/piper_l_with_gripper_description.urdf (robot description, URDF)
Before this commit: robot piper_l, 13 links, 12 joints
Links:
- link link6: mass 0.007 -> 0.00613114124

File: piper_l/urdf/piper_l_with_left_revo2_description.urdf (robot description, URDF)
Before this commit: robot piper_l, 31 links, 30 joints
Links:
- link link6: mass 0.007 -> 0.00613114124

File: piper_l/urdf/piper_l_with_right_revo2_description.urdf (robot description, URDF)
Before this commit: robot piper_l, 31 links, 30 joints
Links:
- link link6: mass 0.007 -> 0.00613114124

File: piper_x/urdf/piper_x_description.urdf (robot description, URDF)
Before this commit: robot piper_x, 8 links, 7 joints
Links:
- link link6: mass 0.007 -> 0.00613114124

File: piper_x/urdf/piper_x_with_gripper_description.urdf (robot description, URDF)
Before this commit: robot piper_x, 13 links, 12 joints
Links:
- link link6: mass 0.007 -> 0.00613114124
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
Commit message: fix(urdf): 调整 Nero J6 关节限位为 -42° 至 50°
修正 Nero 基础模型 J6 限位，各末端 xacro 通过引用同步生效。

---

fix(urdf): adjust Nero J6 joint limits to -42 to 50 degrees

Update the Nero base model J6 limits, inherited by end-effector xacros.

File: nero/urdf/nero_description.urdf (robot description, URDF)
Before this commit: robot nero, 9 links, 8 joints
Joints:
- joint joint6: limit lower=-0.73 upper=0.95 effort=100 velocity=5 -> lower=-0.7330383 upper=0.8726646 effort=100 velocity=5

Commit message: fix(urdf): 同步 Nero 各末端模型 J6 关节限位
将 Nero 基础、法兰、夹爪及左右 Revo2 模型的 J6 限位统一为 -42° 至 50°，保留分支网格路径。

---

fix(urdf): sync Nero J6 limits across end-effector models

Set J6 limits to -42 to 50 degrees for Nero base, flange, gripper and both Revo2 models while preserving branch-specific mesh paths.

File: nero/urdf/nero_description.urdf (robot description, URDF)
Before this commit: robot nero, 9 links, 8 joints
Joints:
- joint joint6: limit lower=-0.73 upper=0.95 effort=100 velocity=5 -> lower=-0.7330383 upper=0.8726646 effort=100 velocity=5

File: nero/urdf/nero_with_flange_description.urdf (robot description, URDF)
Before this commit: robot nero, 10 links, 9 joints
Joints:
- joint joint6: limit lower=-0.73 upper=0.95 effort=100 velocity=5 -> lower=-0.7330383 upper=0.8726646 effort=100 velocity=5

File: nero/urdf/nero_with_gripper_description.urdf (robot description, URDF)
Before this commit: robot nero, 14 links, 13 joints
Joints:
- joint joint6: limit lower=-0.73 upper=0.95 effort=100 velocity=5 -> lower=-0.7330383 upper=0.8726646 effort=100 velocity=5

File: nero/urdf/nero_with_left_revo2_description.urdf (robot description, URDF)
Before this commit: robot nero, 32 links, 31 joints
Joints:
- joint joint6: limit lower=-0.73 upper=0.95 effort=100 velocity=5 -> lower=-0.7330383 upper=0.8726646 effort=100 velocity=5

File: nero/urdf/nero_with_right_revo2_description.urdf (robot description, URDF)
Before this commit: robot nero, 32 links, 31 joints
Joints:
- joint joint6: limit lower=-0.73 upper=0.95 effort=100 velocity=5 -> lower=-0.7330383 upper=0.8726646 effort=100 velocity=5
