Commit message: feat(gripper): add single-DOF gripper joint with mimic finger links
Add a virtual prismatic gripper joint (0–0.1 m opening width) to all
agx_gripper URDF models (nero, piper, piper_h, piper_l, piper_x).
Drive gripper_link1 and gripper_link2 via mimic (×0.5 / ×−0.5) so
visualization and planning only require one controllable DOF.

File: nero/urdf/nero_with_gripper_description.urdf (robot description, URDF)
Before this commit: robot nero, 13 links, 12 joints
Links:
- added link gripper_link
Joints:
- added joint gripper: type prismatic, parent gripper_base, child gripper_link, origin xyz=0 0 0 rpy=0 0 0, axis 0 0 1, limit lower=0 upper=0.1 effort=10 velocity=3
- joint gripper_joint1: mimic (none) -> joint=gripper multiplier=0.5 offset=0.0
- joint gripper_joint2: mimic (none) -> joint=gripper multiplier=-0.5 offset=0.0

File: piper/urdf/piper_with_gripper_description.urdf (robot description, URDF)
Before this commit: robot piper, 11 links, 10 joints
Links:
- added link gripper_link
Joints:
- added joint gripper: type prismatic, parent gripper_base, child gripper_link, origin xyz=0 0 0 rpy=0 0 0, axis 0 0 1, limit lower=0 upper=0.1 effort=10 velocity=3
- joint gripper_joint1: mimic (none) -> joint=gripper multiplier=0.5 offset=0.0
- joint gripper_joint2: mimic (none) -> joint=gripper multiplier=-0.5 offset=0.0

File: piper_h/urdf/piper_h_with_gripper_description.urdf (robot description, URDF)
Before this commit: robot piper_h, 11 links, 10 joints
Links:
- added link gripper_link
Joints:
- added joint gripper: type prismatic, parent gripper_base, child gripper_link, origin xyz=0 0 0 rpy=0 0 0, axis 0 0 1, limit lower=0 upper=0.1 effort=10 velocity=3
- joint gripper_joint1: mimic (none) -> joint=gripper multiplier=0.5 offset=0.0
- joint gripper_joint2: mimic (none) -> joint=gripper multiplier=-0.5 offset=0.0

File: piper_l/urdf/piper_l_with_gripper_description.urdf (robot description, URDF)
Before this commit: robot piper_l, 11 links, 10 joints
Links:
- added link gripper_link
Joints:
- added joint gripper: type prismatic, parent gripper_base, child gripper_link, origin xyz=0 0 0 rpy=0 0 0, axis 0 0 1, limit lower=0 upper=0.1 effort=10 velocity=3
- joint gripper_joint1: mimic (none) -> joint=gripper multiplier=0.5 offset=0.0
- joint gripper_joint2: mimic (none) -> joint=gripper multiplier=-0.5 offset=0.0

File: piper_x/urdf/piper_x_with_gripper_description.urdf (robot description, URDF)
Before this commit: robot piper_x, 11 links, 10 joints
Links:
- added link gripper_link
Joints:
- added joint gripper: type prismatic, parent gripper_base, child gripper_link, origin xyz=0 0 0 rpy=0 0 0, axis 0 0 1, limit lower=0 upper=0.1 effort=10 velocity=3
- joint gripper_joint1: mimic (none) -> joint=gripper multiplier=0.5 offset=0.0
- joint gripper_joint2: mimic (none) -> joint=gripper multiplier=-0.5 offset=0.0

Commit message: feat(urdf): 更新 Piper/Nero 法兰与末端执行器模型
- Piper / Piper H/L/X：新增独立 flange_link（link6 → flange_link → 夹爪/Revo2），更新法兰与夹爪底座 mesh 及惯性参数。
- Piper 夹爪：gripper_base 挂载偏移 0.0045 m，指爪关节原点 Z 调整为 0.138；移除旧版 gripper_base mesh。
- Piper Revo2：hand_base_joint Z 偏移 0.008 → 0.0105 m，同步 flange_link 惯性参数。
- Nero 法兰：gripper_flange / revo2_flange 更新 mesh 与惯性参数，link7 安装位 X 偏移 0.032 → 0.031 m。
- Nero 夹爪：gripper_base 挂载偏移 0.0055 → 0.006 m，指爪关节原点 Z 调整为 0.138；移除 gripper_base_with_flange 资源。

---

feat(urdf): refresh Piper/Nero flange and end-effector models

- Piper / Piper H/L/X: add standalone flange_link (link6 → flange_link → gripper/Revo2); update flange and gripper-base meshes and inertial params.
- Piper gripper: mount gripper_base with 0.0045 m Z offset; set finger joint origin Z to 0.138; remove legacy gripper_base mesh variants.
- Piper Revo2: update hand_base_joint Z offset from 0.008 to 0.0105 m; sync flange_link inertial parameters.
- Nero flanges: refresh gripper_flange / revo2_flange meshes and inertial params; adjust link7 mount X offset from 0.032 to 0.031 m.
- Nero gripper: update gripper_base mount offset from 0.0055 to 0.006 m; set finger joint origin Z to 0.138; remove gripper_base_with_flange assets.

File: nero/urdf/nero_with_gripper_description.urdf (robot description, URDF)
Before this commit: robot nero, 14 links, 13 joints
Joints:
- joint gripper_base_joint: origin xyz=0 0 0.0055 rpy=0 0 0 -> xyz=0 0 0.006 rpy=0 0 0
- joint gripper_flange_joint: origin xyz=0.032 0 -0.0235 rpy=-1.5708 0 -1.5708 -> xyz=0.031 0 -0.0235 rpy=-1.5708 0 -1.5708
- joint gripper_joint1: origin xyz=0 0 0.1358 rpy=1.5707963 0 3.1415926 -> xyz=0 0 0.138 rpy=1.5707963 0 3.1415926
- joint gripper_joint2: origin xyz=0 0 0.1358 rpy=1.5707963 0 0 -> xyz=0 0 0.138 rpy=1.5707963 0 0

File: nero/urdf/nero_with_gripper_flange_description.urdf (robot description, URDF)
Before this commit: robot nero, 10 links, 9 joints
Joints:
- joint gripper_flange_joint: origin xyz=0.032 0 -0.0235 rpy=-1.5708 0 -1.5708 -> xyz=0.031 0 -0.0235 rpy=-1.5708 0 -1.5708

File: nero/urdf/nero_with_left_revo2_description.urdf (robot description, URDF)
Before this commit: robot nero, 32 links, 31 joints
Joints:
- joint revo2_flange_joint: origin xyz=0.032 0 -0.0235 rpy=-1.5708 0 -1.5708 -> xyz=0.031 0 -0.0235 rpy=-1.5708 0 -1.5708

File: nero/urdf/nero_with_revo2_flange_description.urdf (robot description, URDF)
Before this commit: robot nero, 10 links, 9 joints
Joints:
- joint revo2_flange_joint: origin xyz=0.032 0 -0.0235 rpy=-1.5708 0 -1.5708 -> xyz=0.031 0 -0.0235 rpy=-1.5708 0 -1.5708

File: nero/urdf/nero_with_right_revo2_description.urdf (robot description, URDF)
Before this commit: robot nero, 32 links, 31 joints
Joints:
- joint revo2_flange_joint: origin xyz=0.032 0 -0.0235 rpy=-1.5708 0 -1.5708 -> xyz=0.031 0 -0.0235 rpy=-1.5708 0 -1.5708

File: piper/urdf/piper_with_gripper_description.urdf (robot description, URDF)
Before this commit: robot piper, 12 links, 11 joints
Links:
- added link flange_link, mass 0.04; collision mesh filename=../meshes/flange.stl; visual mesh filename=../meshes/dae/flange.dae
Joints:
- added joint flange_joint: type fixed, parent link6, child flange_link, origin xyz=0 0 0 rpy=0 0 0
- joint gripper_base_joint: origin xyz=0 0 0 rpy=0 0 0 -> xyz=0 0 0.0045 rpy=0 0 0; parent link6 -> flange_link
- joint gripper_joint1: origin xyz=0 0 0.1358 rpy=1.5707963 0 0 -> xyz=0 0 0.138 rpy=1.5707963 0 0
- joint gripper_joint2: origin xyz=0 0 0.1358 rpy=1.5707963 0 -3.1415926 -> xyz=0 0 0.138 rpy=1.5707963 0 -3.1415926

File: piper/urdf/piper_with_left_revo2_description.urdf (robot description, URDF)
Before this commit: robot piper, 31 links, 30 joints
Links:
- link flange_link: mass 0.001 -> 0.04
Joints:
- joint hand_base_joint: origin xyz=0.0 0.0 0.008 rpy=0 0 0 -> xyz=0.0 0.0 0.0105 rpy=0 0 0

File: piper/urdf/piper_with_right_revo2_description.urdf (robot description, URDF)
Before this commit: robot piper, 31 links, 30 joints
Links:
- link flange_link: mass 0.001 -> 0.04
Joints:
- joint hand_base_joint: origin xyz=0.0 0.0 0.008 rpy=0 0 0 -> xyz=0.0 0.0 0.0105 rpy=0 0 0

File: piper_h/urdf/piper_h_with_gripper_description.urdf (robot description, URDF)
Before this commit: robot piper_h, 12 links, 11 joints
Links:
- added link flange_link, mass 0.04; collision mesh filename=../meshes/flange.stl; visual mesh filename=../meshes/dae/flange.dae
Joints:
- added joint flange_joint: type fixed, parent link6, child flange_link, origin xyz=0 0 0 rpy=0 0 0
- joint gripper_base_joint: origin xyz=0 0 0 rpy=0 0 0 -> xyz=0 0 0.0045 rpy=0 0 0; parent link6 -> flange_link
- joint gripper_joint1: origin xyz=0 0 0.1358 rpy=1.5707963 0 0 -> xyz=0 0 0.138 rpy=1.5707963 0 0
- joint gripper_joint2: origin xyz=0 0 0.1358 rpy=1.5707963 0 -3.1415926 -> xyz=0 0 0.138 rpy=1.5707963 0 -3.1415926

File: piper_h/urdf/piper_h_with_left_revo2_description.urdf (robot description, URDF)
Before this commit: robot piper_h, 31 links, 30 joints
Links:
- link flange_link: mass 0.001 -> 0.04
Joints:
- joint hand_base_joint: origin xyz=0.0 0.0 0.008 rpy=0 0 0 -> xyz=0.0 0.0 0.0105 rpy=0 0 0

File: piper_h/urdf/piper_h_with_right_revo2_description.urdf (robot description, URDF)
Before this commit: robot piper_h, 31 links, 30 joints
Links:
- link flange_link: mass 0.001 -> 0.04
Joints:
- joint hand_base_joint: origin xyz=0.0 0.0 0.008 rpy=0 0 0 -> xyz=0.0 0.0 0.0105 rpy=0 0 0

File: piper_l/urdf/piper_l_with_gripper_description.urdf (robot description, URDF)
Before this commit: robot piper_l, 12 links, 11 joints
Links:
- added link flange_link, mass 0.04; collision mesh filename=../meshes/flange.stl; visual mesh filename=../meshes/dae/flange.dae
Joints:
- added joint flange_joint: type fixed, parent link6, child flange_link, origin xyz=0 0 0 rpy=0 0 0
- joint gripper_base_joint: origin xyz=0 0 0 rpy=0 0 0 -> xyz=0 0 0.0045 rpy=0 0 0; parent link6 -> flange_link
- joint gripper_joint1: origin xyz=0 0 0.1358 rpy=1.5707963 0 0 -> xyz=0 0 0.138 rpy=1.5707963 0 0
- joint gripper_joint2: origin xyz=0 0 0.1358 rpy=1.5707963 0 -3.1415926 -> xyz=0 0 0.138 rpy=1.5707963 0 -3.1415926

File: piper_l/urdf/piper_l_with_left_revo2_description.urdf (robot description, URDF)
Before this commit: robot piper_l, 31 links, 30 joints
Links:
- link flange_link: mass 0.001 -> 0.04
Joints:
- joint hand_base_joint: origin xyz=0.0 0.0 0.008 rpy=0 0 0 -> xyz=0.0 0.0 0.0105 rpy=0 0 0

File: piper_l/urdf/piper_l_with_right_revo2_description.urdf (robot description, URDF)
Before this commit: robot piper_l, 31 links, 30 joints
Links:
- link flange_link: mass 0.001 -> 0.04
Joints:
- joint hand_base_joint: origin xyz=0.0 0.0 0.008 rpy=0 0 0 -> xyz=0.0 0.0 0.0105 rpy=0 0 0

File: piper_x/urdf/piper_x_with_gripper_description.urdf (robot description, URDF)
Before this commit: robot piper_x, 12 links, 11 joints
Links:
- added link flange_link, mass 0.04; collision mesh filename=../meshes/flange.stl; visual mesh filename=../meshes/dae/flange.dae
Joints:
- added joint flange_joint: type fixed, parent link6, child flange_link, origin xyz=0 0 0 rpy=0 0 0
- joint gripper_base_joint: origin xyz=0 0 0 rpy=0 0 1.5707963 -> xyz=0 0 0.0045 rpy=0 0 1.5707963; parent link6 -> flange_link
- joint gripper_joint1: origin xyz=0 0 0.1358 rpy=1.5707963 0 0 -> xyz=0 0 0.138 rpy=1.5707963 0 0
- joint gripper_joint2: origin xyz=0 0 0.1358 rpy=1.5707963 0 -3.1415926 -> xyz=0 0 0.138 rpy=1.5707963 0 -3.1415926

File: piper_x/urdf/piper_x_with_left_revo2_description.urdf (robot description, URDF)
Before this commit: robot piper_x, 31 links, 30 joints
Links:
- link flange_link: mass 0.001 -> 0.04
Joints:
- joint hand_base_joint: origin xyz=0.0 0.0 0.008 rpy=0 0 0 -> xyz=0.0 0.0 0.0105 rpy=0 0 0

File: piper_x/urdf/piper_x_with_right_revo2_description.urdf (robot description, URDF)
Before this commit: robot piper_x, 31 links, 30 joints
Links:
- link flange_link: mass 0.001 -> 0.04
Joints:
- joint hand_base_joint: origin xyz=0.0 0.0 0.008 rpy=0 0 0 -> xyz=0.0 0.0 0.0105 rpy=0 0 0
