Commit message: fix(urdf): 同步 Piper/Nero 末端连杆质量与惯量
- 同步 main 提交 9f45f05 的 link6/link7 质量与惯量修正
- 更新基础模型及夹爪、Revo2 和法兰组合的 22 个 URDF
- 保留当前分支的网格路径和目录结构

---

fix(urdf): sync Piper/Nero end-link mass and inertia

- Sync the link6/link7 mass and inertia corrections from main commit 9f45f05
- Update 22 URDF files covering base models, grippers, Revo2 hands and flange combinations
- Preserve branch-specific mesh paths and directory structure

File: nero/urdf/nero_with_gripper_description.urdf (robot description, URDF)
Before this commit: robot nero, 14 links, 13 joints
Links:
- link link7: mass 0.000001 -> 0.001

File: nero/urdf/nero_with_gripper_flange_description.urdf (robot description, URDF)
Before this commit: robot nero, 10 links, 9 joints
Links:
- link link7: mass 0.000001 -> 0.001

File: nero/urdf/nero_with_left_revo2_description.urdf (robot description, URDF)
Before this commit: robot nero, 32 links, 31 joints
Links:
- link link7: mass 0.000001 -> 0.001

File: nero/urdf/nero_with_revo2_flange_description.urdf (robot description, URDF)
Before this commit: robot nero, 10 links, 9 joints
Links:
- link link7: mass 0.000001 -> 0.001

File: nero/urdf/nero_with_right_revo2_description.urdf (robot description, URDF)
Before this commit: robot nero, 32 links, 31 joints
Links:
- link link7: mass 0.000001 -> 0.001

File: piper/urdf/piper_with_gripper_description.urdf (robot description, URDF)
Before this commit: robot piper, 13 links, 12 joints
Links:
- link link6: mass 0.007 -> 0.00613114124

File: piper/urdf/piper_with_left_revo2_description.urdf (robot description, URDF)
Before this commit: robot piper, 31 links, 30 joints
Links:
- link link6: mass 0.007 -> 0.00613114124

File: piper/urdf/piper_with_right_revo2_description.urdf (robot description, URDF)
Before this commit: robot piper, 31 links, 30 joints
Links:
- link link6: mass 0.007 -> 0.00613114124

File: piper_h/urdf/piper_h_with_gripper_description.urdf (robot description, URDF)
Before this commit: robot piper_h, 13 links, 12 joints
Links:
- link link6: mass 0.007 -> 0.00613114124

File: piper_h/urdf/piper_h_with_left_revo2_description.urdf (robot description, URDF)
Before this commit: robot piper_h, 31 links, 30 joints
Links:
- link link6: mass 0.007 -> 0.00613114124

File: piper_h/urdf/piper_h_with_right_revo2_description.urdf (robot description, URDF)
Before this commit: robot piper_h, 31 links, 30 joints
Links:
- link link6: mass 0.007 -> 0.00613114124

File: piper_l/urdf/piper_l_with_gripper_description.urdf (robot description, URDF)
Before this commit: robot piper_l, 13 links, 12 joints
Links:
- link link6: mass 0.007 -> 0.00613114124

File: piper_l/urdf/piper_l_with_left_revo2_description.urdf (robot description, URDF)
Before this commit: robot piper_l, 31 links, 30 joints
Links:
- link link6: mass 0.007 -> 0.00613114124

File: piper_l/urdf/piper_l_with_right_revo2_description.urdf (robot description, URDF)
Before this commit: robot piper_l, 31 links, 30 joints
Links:
- link link6: mass 0.007 -> 0.00613114124

File: piper_x/urdf/piper_x_with_gripper_description.urdf (robot description, URDF)
Before this commit: robot piper_x, 13 links, 12 joints
Links:
- link link6: mass 0.007 -> 0.00613114124

File: piper_x/urdf/piper_x_with_left_revo2_description.urdf (robot description, URDF)
Before this commit: robot piper_x, 31 links, 30 joints
Links:
- link link6: mass 0.007 -> 0.00613114124

File: piper_x/urdf/piper_x_with_right_revo2_description.urdf (robot description, URDF)
Before this commit: robot piper_x, 31 links, 30 joints
Links:
- link link6: mass 0.007 -> 0.00613114124
