Commit message: Add mimic joint to nero gripper so both fingers track one DOF
The two gripper fingers are driven by a single motor (mechanically
coupled), but the URDF modeled them as two independent prismatic joints.
This adds a <mimic> tag so gripper_joint2 follows gripper_joint1 (x-1.0),
matching the real hardware and letting robot_state_publisher derive the
second finger from a single published value.

File: nero/urdf/nero_with_gripper_description.xacro (robot description, xacro)
@@ -79,4 +79,5 @@
         <axis xyz="0 0 -1"/>
         <limit lower="-0.05" upper="0" effort="10" velocity="3"/>
+        <mimic joint="gripper_joint1" multiplier="-1.0" offset="0.0"/>
     </joint>
 </robot>

Commit message: feat(gripper): add single-DOF gripper joint with mimic finger links
Add a virtual prismatic gripper joint (0–0.1 m opening width) to all
agx_gripper URDF models (nero, piper, piper_h, piper_l, piper_x).
Drive gripper_link1 and gripper_link2 via mimic (×0.5 / ×−0.5) so
visualization and planning only require one controllable DOF.

File: nero/urdf/nero_with_gripper_description.xacro (robot description, xacro)
@@ -28,4 +28,12 @@
         <child link="gripper_base"/>
     </joint>
+    <link name="gripper_link"/>
+    <joint name="gripper" type="prismatic">
+        <origin xyz="0 0 0" rpy="0 0 0"/>
+        <parent link="gripper_base"/>
+        <child link="gripper_link"/>
+        <axis xyz="0 0 1"/>
+        <limit lower="0" upper="0.1" effort="10" velocity="3"/>
+    </joint>
     <link name="gripper_link1">
         <inertial>
@@ -53,4 +61,5 @@
         <axis xyz="0 0 1"/>
         <limit lower="0" upper="0.05" effort="10" velocity="3"/>
+        <mimic joint="gripper" multiplier="0.5" offset="0.0"/>
     </joint>
     <link name="gripper_link2">
@@ -79,4 +88,5 @@
         <axis xyz="0 0 -1"/>
         <limit lower="-0.05" upper="0" effort="10" velocity="3"/>
+        <mimic joint="gripper" multiplier="-0.5" offset="0.0"/>
     </joint>
 </robot>

File: piper/urdf/piper_with_gripper_description.xacro (robot description, xacro)
@@ -28,4 +28,12 @@
         <child link="gripper_base"/>
     </joint>
+    <link name="gripper_link"/>
+    <joint name="gripper" type="prismatic">
+        <origin xyz="0 0 0" rpy="0 0 0"/>
+        <parent link="gripper_base"/>
+        <child link="gripper_link"/>
+        <axis xyz="0 0 1"/>
+        <limit lower="0" upper="0.1" effort="10" velocity="3"/>
+    </joint>
     <link name="gripper_link1">
         <inertial>
@@ -53,4 +61,5 @@
         <axis xyz="0 0 1"/>
         <limit lower="0" upper="0.05" effort="10" velocity="3"/>
+        <mimic joint="gripper" multiplier="0.5" offset="0.0"/>
     </joint>
     <link name="gripper_link2">
@@ -79,4 +88,5 @@
         <axis xyz="0 0 -1"/>
         <limit lower="-0.05" upper="0" effort="10" velocity="3"/>
+        <mimic joint="gripper" multiplier="-0.5" offset="0.0"/>
     </joint>
 </robot>

File: piper_h/urdf/piper_h_with_gripper_description.xacro (robot description, xacro)
@@ -28,4 +28,12 @@
         <child link="gripper_base"/>
     </joint>
+    <link name="gripper_link"/>
+    <joint name="gripper" type="prismatic">
+        <origin xyz="0 0 0" rpy="0 0 0"/>
+        <parent link="gripper_base"/>
+        <child link="gripper_link"/>
+        <axis xyz="0 0 1"/>
+        <limit lower="0" upper="0.1" effort="10" velocity="3"/>
+    </joint>
     <link name="gripper_link1">
         <inertial>
@@ -53,4 +61,5 @@
         <axis xyz="0 0 1"/>
         <limit lower="0" upper="0.05" effort="10" velocity="3"/>
+        <mimic joint="gripper" multiplier="0.5" offset="0.0"/>
     </joint>
     <link name="gripper_link2">
@@ -79,4 +88,5 @@
         <axis xyz="0 0 -1"/>
         <limit lower="-0.05" upper="0" effort="10" velocity="3"/>
+        <mimic joint="gripper" multiplier="-0.5" offset="0.0"/>
     </joint>
 </robot>

File: piper_l/urdf/piper_l_with_gripper_description.xacro (robot description, xacro)
@@ -28,4 +28,12 @@
         <child link="gripper_base"/>
     </joint>
+    <link name="gripper_link"/>
+    <joint name="gripper" type="prismatic">
+        <origin xyz="0 0 0" rpy="0 0 0"/>
+        <parent link="gripper_base"/>
+        <child link="gripper_link"/>
+        <axis xyz="0 0 1"/>
+        <limit lower="0" upper="0.1" effort="10" velocity="3"/>
+    </joint>
     <link name="gripper_link1">
         <inertial>
@@ -53,4 +61,5 @@
         <axis xyz="0 0 1"/>
         <limit lower="0" upper="0.05" effort="10" velocity="3"/>
+        <mimic joint="gripper" multiplier="0.5" offset="0.0"/>
     </joint>
     <link name="gripper_link2">
@@ -79,4 +88,5 @@
         <axis xyz="0 0 -1"/>
         <limit lower="-0.05" upper="0" effort="10" velocity="3"/>
+        <mimic joint="gripper" multiplier="-0.5" offset="0.0"/>
     </joint>
 </robot>

File: piper_x/urdf/piper_x_with_gripper_description.xacro (robot description, xacro)
@@ -28,4 +28,12 @@
         <child link="gripper_base"/>
     </joint>
+    <link name="gripper_link"/>
+    <joint name="gripper" type="prismatic">
+        <origin xyz="0 0 0" rpy="0 0 0"/>
+        <parent link="gripper_base"/>
+        <child link="gripper_link"/>
+        <axis xyz="0 0 1"/>
+        <limit lower="0" upper="0.1" effort="10" velocity="3"/>
+    </joint>
     <link name="gripper_link1">
         <inertial>
@@ -53,4 +61,5 @@
         <axis xyz="0 0 1"/>
         <limit lower="0" upper="0.05" effort="10" velocity="3"/>
+        <mimic joint="gripper" multiplier="0.5" offset="0.0"/>
     </joint>
     <link name="gripper_link2">
@@ -79,4 +88,5 @@
         <axis xyz="0 0 -1"/>
         <limit lower="-0.05" upper="0" effort="10" velocity="3"/>
+        <mimic joint="gripper" multiplier="-0.5" offset="0.0"/>
     </joint>
 </robot>
