Commit message: feat(urdf): 更新 Piper/Nero 法兰与末端执行器模型
- Piper / Piper H/L/X：新增独立 flange_link（link6 → flange_link → 夹爪/Revo2），更新法兰与夹爪底座 mesh 及惯性参数。
- Piper 夹爪：gripper_base 挂载偏移 0.0045 m，指爪关节原点 Z 调整为 0.138；移除旧版 gripper_base mesh。
- Piper Revo2：hand_base_joint Z 偏移 0.008 → 0.0105 m，同步 flange_link 惯性参数。
- Nero 法兰：gripper_flange / revo2_flange 更新 mesh 与惯性参数，link7 安装位 X 偏移 0.032 → 0.031 m。
- Nero 夹爪：gripper_base 挂载偏移 0.0055 → 0.006 m，指爪关节原点 Z 调整为 0.138；移除 gripper_base_with_flange 资源。

---

feat(urdf): refresh Piper/Nero flange and end-effector models

- Piper / Piper H/L/X: add standalone flange_link (link6 → flange_link → gripper/Revo2); update flange and gripper-base meshes and inertial params.
- Piper gripper: mount gripper_base with 0.0045 m Z offset; set finger joint origin Z to 0.138; remove legacy gripper_base mesh variants.
- Piper Revo2: update hand_base_joint Z offset from 0.008 to 0.0105 m; sync flange_link inertial parameters.
- Nero flanges: refresh gripper_flange / revo2_flange meshes and inertial params; adjust link7 mount X offset from 0.032 to 0.031 m.
- Nero gripper: update gripper_base mount offset from 0.0055 to 0.006 m; set finger joint origin Z to 0.138; remove gripper_base_with_flange assets.

File: nero/urdf/nero_with_gripper_description.xacro (robot description, xacro)
@@ -24,5 +24,5 @@
     </link>
     <joint name="gripper_base_joint" type="fixed">
-        <origin xyz="0 0 0.0055" rpy="0 0 0"/>
+        <origin xyz="0 0 0.006" rpy="0 0 0"/>
         <parent link="gripper_flange"/>
         <child link="gripper_base"/>
@@ -56,5 +56,5 @@
     </link>
     <joint name="gripper_joint1" type="prismatic">
-        <origin xyz="0 0 0.1358" rpy="1.5707963 0 3.1415926"/>
+        <origin xyz="0 0 0.138" rpy="1.5707963 0 3.1415926"/>
         <parent link="gripper_base"/>
         <child link="gripper_link1"/>
@@ -83,5 +83,5 @@
     </link>
     <joint name="gripper_joint2" type="prismatic">
-        <origin xyz="0 0 0.1358" rpy="1.5707963 0 0"/>
+        <origin xyz="0 0 0.138" rpy="1.5707963 0 0"/>
         <parent link="gripper_base"/>
         <child link="gripper_link2"/>

File: nero/urdf/nero_with_gripper_flange_description.xacro (robot description, xacro)
@@ -6,7 +6,7 @@
     <link name="gripper_flange">
         <inertial>
-            <origin xyz="0.0 0.0 -0.00032" rpy="0 0 0"/>
+            <origin xyz="0.000253201 -0.000322696 -0.010082901" rpy="0 0 0"/>
             <mass value="0.04771096"/>
-            <inertia ixx="2.697e-05" ixy="0" ixz="0" iyy="4.311e-05" iyz="0" izz="2.479e-05"/>
+            <inertia ixx="36.14107e-06" ixy="0" ixz="0" iyy="17.824164e-06" iyz="0" izz="26.95944e-06"/>
         </inertial>
         <visual>
@@ -24,5 +24,5 @@
     </link>
     <joint name="gripper_flange_joint" type="fixed">
-        <origin xyz="0.032 0 -0.0235" rpy="-1.5708 0 -1.5708"/>
+        <origin xyz="0.031 0 -0.0235" rpy="-1.5708 0 -1.5708"/>
         <parent link="link7"/>
         <child link="gripper_flange"/>

File: nero/urdf/nero_with_revo2_flange_description.xacro (robot description, xacro)
@@ -6,7 +6,7 @@
     <link name="revo2_flange">
         <inertial>
-            <origin xyz="0.0 0.0 -0.00032" rpy="0 0 0"/>
+            <origin xyz="0.000253201 -0.000322696 -0.010082901" rpy="0 0 0"/>
             <mass value="0.04771096"/>
-            <inertia ixx="2.697e-05" ixy="0" ixz="0" iyy="4.311e-05" iyz="0" izz="2.479e-05"/>
+            <inertia ixx="36.14107e-06" ixy="0" ixz="0" iyy="17.824164e-06" iyz="0" izz="26.95944e-06"/>
         </inertial>
         <visual>
@@ -24,5 +24,5 @@
     </link>
     <joint name="revo2_flange_joint" type="fixed">
-        <origin xyz="0.032 0 -0.0235" rpy="-1.5708 0 -1.5708"/>
+        <origin xyz="0.031 0 -0.0235" rpy="-1.5708 0 -1.5708"/>
         <parent link="link7"/>
         <child link="revo2_flange"/>

File: piper/urdf/piper_with_gripper_description.xacro (robot description, xacro)
@@ -4,4 +4,28 @@
 <robot xmlns:xacro="http://www.ros.org/wiki/xacro" name="piper">
 <xacro:include filename="$(find agx_arm_description)/agx_arm_urdf/piper/urdf/piper_description.urdf"/>
+    <link name="flange_link">
+        <inertial>
+            <origin xyz="1.151691e-03 0.782428e-03 4.798051e-03" rpy="0 0 0"/>
+            <mass value="0.04"/>
+            <inertia ixx="9.935389e-06" ixy="0.0" ixz="0.0" iyy="10.508003e-06" iyz="0.0" izz="19.652873e-06"/>
+        </inertial>
+        <visual>
+            <origin xyz="0 0 0" rpy="0 0 0"/>
+            <geometry>
+                <mesh filename="package://agx_arm_description/agx_arm_urdf/piper/meshes/dae/flange.dae"/>
+            </geometry>
+        </visual>
+        <collision>
+            <origin xyz="0 0 0" rpy="0 0 0"/>
+            <geometry>
+                <mesh filename="package://agx_arm_description/agx_arm_urdf/piper/meshes/flange.stl"/>
+            </geometry>
+        </collision>
+    </link>
+    <joint name="flange_joint" type="fixed">
+        <origin xyz="0 0 0" rpy="0 0 0"/>
+        <parent link="link6"/>
+        <child link="flange_link"/>
+    </joint>
     <link name="gripper_base">
         <inertial>
@@ -24,6 +48,6 @@
     </link>
     <joint name="gripper_base_joint" type="fixed">
-        <origin xyz="0 0 0" rpy="0 0 0"/>
-        <parent link="link6"/>
+        <origin xyz="0 0 0.0045" rpy="0 0 0"/>
+        <parent link="flange_link"/>
         <child link="gripper_base"/>
     </joint>
@@ -56,5 +80,5 @@
     </link>
     <joint name="gripper_joint1" type="prismatic">
-        <origin xyz="0 0 0.1358" rpy="1.5707963 0 0"/>
+        <origin xyz="0 0 0.138" rpy="1.5707963 0 0"/>
         <parent link="gripper_base"/>
         <child link="gripper_link1"/>
@@ -83,5 +107,5 @@
     </link>
     <joint name="gripper_joint2" type="prismatic">
-        <origin xyz="0 0 0.1358" rpy="1.5707963 0 -3.1415926"/>
+        <origin xyz="0 0 0.138" rpy="1.5707963 0 -3.1415926"/>
         <parent link="gripper_base"/>
         <child link="gripper_link2"/>

File: piper/urdf/piper_with_left_revo2_description.xacro (robot description, xacro)
@@ -8,7 +8,7 @@
     <link name="flange_link">
         <inertial>
-            <origin xyz="0.0 0.0 0.004" rpy="0 0 0"/>
-            <mass value="0.001"/>
-            <inertia ixx="0.00000001" ixy="0.00000000" ixz="0.00000000" iyy="0.00000001" iyz="0.00000000" izz="0.00000001"/>
+            <origin xyz="1.151691e-03 0.782428e-03 4.798051e-03" rpy="0 0 0"/>
+            <mass value="0.04"/>
+            <inertia ixx="9.935389e-06" ixy="0.0" ixz="0.0" iyy="10.508003e-06" iyz="0.0" izz="19.652873e-06"/>
         </inertial>
         <visual>
@@ -31,5 +31,5 @@
     </joint>
     <joint name="hand_base_joint" type="fixed">
-        <origin xyz="0.0 0.0 0.008" rpy="0 0 0"/>
+        <origin xyz="0.0 0.0 0.0105" rpy="0 0 0"/>
         <parent link="flange_link"/>
         <child link="left_base_link"/>

File: piper/urdf/piper_with_right_revo2_description.xacro (robot description, xacro)
@@ -8,7 +8,7 @@
     <link name="flange_link">
         <inertial>
-            <origin xyz="0.0 0.0 0.004" rpy="0 0 0"/>
-            <mass value="0.001"/>
-            <inertia ixx="0.00000001" ixy="0.00000000" ixz="0.00000000" iyy="0.00000001" iyz="0.00000000" izz="0.00000001"/>
+            <origin xyz="1.151691e-03 0.782428e-03 4.798051e-03" rpy="0 0 0"/>
+            <mass value="0.04"/>
+            <inertia ixx="9.935389e-06" ixy="0.0" ixz="0.0" iyy="10.508003e-06" iyz="0.0" izz="19.652873e-06"/>
         </inertial>
         <visual>
@@ -31,5 +31,5 @@
     </joint>
     <joint name="hand_base_joint" type="fixed">
-        <origin xyz="0.0 0.0 0.008" rpy="0 0 0"/>
+        <origin xyz="0.0 0.0 0.0105" rpy="0 0 0"/>
         <parent link="flange_link"/>
         <child link="right_base_link"/>

File: piper_h/urdf/piper_h_with_gripper_description.xacro (robot description, xacro)
@@ -4,4 +4,28 @@
 <robot xmlns:xacro="http://www.ros.org/wiki/xacro" name="piper_h">
 <xacro:include filename="$(find agx_arm_description)/agx_arm_urdf/piper_h/urdf/piper_h_description.urdf"/>
+    <link name="flange_link">
+        <inertial>
+            <origin xyz="1.151691e-03 0.782428e-03 4.798051e-03" rpy="0 0 0"/>
+            <mass value="0.04"/>
+            <inertia ixx="9.935389e-06" ixy="0.0" ixz="0.0" iyy="10.508003e-06" iyz="0.0" izz="19.652873e-06"/>
+        </inertial>
+        <visual>
+            <origin xyz="0 0 0" rpy="0 0 0"/>
+            <geometry>
+                <mesh filename="package://agx_arm_description/agx_arm_urdf/piper_h/meshes/dae/flange.dae"/>
+            </geometry>
+        </visual>
+        <collision>
+            <origin xyz="0 0 0" rpy="0 0 0"/>
+            <geometry>
+                <mesh filename="package://agx_arm_description/agx_arm_urdf/piper_h/meshes/flange.stl"/>
+            </geometry>
+        </collision>
+    </link>
+    <joint name="flange_joint" type="fixed">
+        <origin xyz="0 0 0" rpy="0 0 0"/>
+        <parent link="link6"/>
+        <child link="flange_link"/>
+    </joint>
     <link name="gripper_base">
         <inertial>
@@ -24,6 +48,6 @@
     </link>
     <joint name="gripper_base_joint" type="fixed">
-        <origin xyz="0 0 0" rpy="0 0 0"/>
-        <parent link="link6"/>
+        <origin xyz="0 0 0.0045" rpy="0 0 0"/>
+        <parent link="flange_link"/>
         <child link="gripper_base"/>
     </joint>
@@ -56,5 +80,5 @@
     </link>
     <joint name="gripper_joint1" type="prismatic">
-        <origin xyz="0 0 0.1358" rpy="1.5707963 0 0"/>
+        <origin xyz="0 0 0.138" rpy="1.5707963 0 0"/>
         <parent link="gripper_base"/>
         <child link="gripper_link1"/>
@@ -83,5 +107,5 @@
     </link>
     <joint name="gripper_joint2" type="prismatic">
-        <origin xyz="0 0 0.1358" rpy="1.5707963 0 -3.1415926"/>
+        <origin xyz="0 0 0.138" rpy="1.5707963 0 -3.1415926"/>
         <parent link="gripper_base"/>
         <child link="gripper_link2"/>

File: piper_h/urdf/piper_h_with_left_revo2_description.xacro (robot description, xacro)
@@ -8,7 +8,7 @@
     <link name="flange_link">
         <inertial>
-            <origin xyz="0.0 0.0 0.004" rpy="0 0 0"/>
-            <mass value="0.001"/>
-            <inertia ixx="0.00000001" ixy="0.00000000" ixz="0.00000000" iyy="0.00000001" iyz="0.00000000" izz="0.00000001"/>
+            <origin xyz="1.151691e-03 0.782428e-03 4.798051e-03" rpy="0 0 0"/>
+            <mass value="0.04"/>
+            <inertia ixx="9.935389e-06" ixy="0.0" ixz="0.0" iyy="10.508003e-06" iyz="0.0" izz="19.652873e-06"/>
         </inertial>
         <visual>
@@ -31,5 +31,5 @@
     </joint>
     <joint name="hand_base_joint" type="fixed">
-        <origin xyz="0.0 0.0 0.008" rpy="0 0 0"/>
+        <origin xyz="0.0 0.0 0.0105" rpy="0 0 0"/>
         <parent link="flange_link"/>
         <child link="left_base_link"/>

File: piper_h/urdf/piper_h_with_right_revo2_description.xacro (robot description, xacro)
@@ -8,7 +8,7 @@
     <link name="flange_link">
         <inertial>
-            <origin xyz="0.0 0.0 0.004" rpy="0 0 0"/>
-            <mass value="0.001"/>
-            <inertia ixx="0.00000001" ixy="0.00000000" ixz="0.00000000" iyy="0.00000001" iyz="0.00000000" izz="0.00000001"/>
+            <origin xyz="1.151691e-03 0.782428e-03 4.798051e-03" rpy="0 0 0"/>
+            <mass value="0.04"/>
+            <inertia ixx="9.935389e-06" ixy="0.0" ixz="0.0" iyy="10.508003e-06" iyz="0.0" izz="19.652873e-06"/>
         </inertial>
         <visual>
@@ -31,5 +31,5 @@
     </joint>
     <joint name="hand_base_joint" type="fixed">
-        <origin xyz="0.0 0.0 0.008" rpy="0 0 0"/>
+        <origin xyz="0.0 0.0 0.0105" rpy="0 0 0"/>
         <parent link="flange_link"/>
         <child link="right_base_link"/>

File: piper_l/urdf/piper_l_with_gripper_description.xacro (robot description, xacro)
@@ -4,4 +4,28 @@
 <robot xmlns:xacro="http://www.ros.org/wiki/xacro" name="piper_l">
 <xacro:include filename="$(find agx_arm_description)/agx_arm_urdf/piper_l/urdf/piper_l_description.urdf"/>
+    <link name="flange_link">
+        <inertial>
+            <origin xyz="1.151691e-03 0.782428e-03 4.798051e-03" rpy="0 0 0"/>
+            <mass value="0.04"/>
+            <inertia ixx="9.935389e-06" ixy="0.0" ixz="0.0" iyy="10.508003e-06" iyz="0.0" izz="19.652873e-06"/>
+        </inertial>
+        <visual>
+            <origin xyz="0 0 0" rpy="0 0 0"/>
+            <geometry>
+                <mesh filename="package://agx_arm_description/agx_arm_urdf/piper_l/meshes/dae/flange.dae"/>
+            </geometry>
+        </visual>
+        <collision>
+            <origin xyz="0 0 0" rpy="0 0 0"/>
+            <geometry>
+                <mesh filename="package://agx_arm_description/agx_arm_urdf/piper_l/meshes/flange.stl"/>
+            </geometry>
+        </collision>
+    </link>
+    <joint name="flange_joint" type="fixed">
+        <origin xyz="0 0 0" rpy="0 0 0"/>
+        <parent link="link6"/>
+        <child link="flange_link"/>
+    </joint>
     <link name="gripper_base">
         <inertial>
@@ -24,6 +48,6 @@
     </link>
     <joint name="gripper_base_joint" type="fixed">
-        <origin xyz="0 0 0" rpy="0 0 0"/>
-        <parent link="link6"/>
+        <origin xyz="0 0 0.0045" rpy="0 0 0"/>
+        <parent link="flange_link"/>
         <child link="gripper_base"/>
     </joint>
@@ -56,5 +80,5 @@
     </link>
     <joint name="gripper_joint1" type="prismatic">
-        <origin xyz="0 0 0.1358" rpy="1.5707963 0 0"/>
+        <origin xyz="0 0 0.138" rpy="1.5707963 0 0"/>
         <parent link="gripper_base"/>
         <child link="gripper_link1"/>
@@ -83,5 +107,5 @@
     </link>
     <joint name="gripper_joint2" type="prismatic">
-        <origin xyz="0 0 0.1358" rpy="1.5707963 0 -3.1415926"/>
+        <origin xyz="0 0 0.138" rpy="1.5707963 0 -3.1415926"/>
         <parent link="gripper_base"/>
         <child link="gripper_link2"/>

File: piper_l/urdf/piper_l_with_left_revo2_description.xacro (robot description, xacro)
@@ -8,7 +8,7 @@
     <link name="flange_link">
         <inertial>
-            <origin xyz="0.0 0.0 0.004" rpy="0 0 0"/>
-            <mass value="0.001"/>
-            <inertia ixx="0.00000001" ixy="0.00000000" ixz="0.00000000" iyy="0.00000001" iyz="0.00000000" izz="0.00000001"/>
+            <origin xyz="1.151691e-03 0.782428e-03 4.798051e-03" rpy="0 0 0"/>
+            <mass value="0.04"/>
+            <inertia ixx="9.935389e-06" ixy="0.0" ixz="0.0" iyy="10.508003e-06" iyz="0.0" izz="19.652873e-06"/>
         </inertial>
         <visual>
@@ -31,5 +31,5 @@
     </joint>
     <joint name="hand_base_joint" type="fixed">
-        <origin xyz="0.0 0.0 0.008" rpy="0 0 0"/>
+        <origin xyz="0.0 0.0 0.0105" rpy="0 0 0"/>
         <parent link="flange_link"/>
         <child link="left_base_link"/>

File: piper_l/urdf/piper_l_with_right_revo2_description.xacro (robot description, xacro)
@@ -8,7 +8,7 @@
     <link name="flange_link">
         <inertial>
-            <origin xyz="0.0 0.0 0.004" rpy="0 0 0"/>
-            <mass value="0.001"/>
-            <inertia ixx="0.00000001" ixy="0.00000000" ixz="0.00000000" iyy="0.00000001" iyz="0.00000000" izz="0.00000001"/>
+            <origin xyz="1.151691e-03 0.782428e-03 4.798051e-03" rpy="0 0 0"/>
+            <mass value="0.04"/>
+            <inertia ixx="9.935389e-06" ixy="0.0" ixz="0.0" iyy="10.508003e-06" iyz="0.0" izz="19.652873e-06"/>
         </inertial>
         <visual>
@@ -31,5 +31,5 @@
     </joint>
     <joint name="hand_base_joint" type="fixed">
-        <origin xyz="0.0 0.0 0.008" rpy="0 0 0"/>
+        <origin xyz="0.0 0.0 0.0105" rpy="0 0 0"/>
         <parent link="flange_link"/>
         <child link="right_base_link"/>

File: piper_x/urdf/piper_x_with_gripper_description.xacro (robot description, xacro)
@@ -4,4 +4,28 @@
 <robot xmlns:xacro="http://www.ros.org/wiki/xacro" name="piper_x">
 <xacro:include filename="$(find agx_arm_description)/agx_arm_urdf/piper_x/urdf/piper_x_description.urdf"/>
+    <link name="flange_link">
+        <inertial>
+            <origin xyz="1.151691e-03 0.782428e-03 4.798051e-03" rpy="0 0 0"/>
+            <mass value="0.04"/>
+            <inertia ixx="9.935389e-06" ixy="0.0" ixz="0.0" iyy="10.508003e-06" iyz="0.0" izz="19.652873e-06"/>
+        </inertial>
+        <visual>
+            <origin xyz="0 0 0" rpy="0 0 0"/>
+            <geometry>
+                <mesh filename="package://agx_arm_description/agx_arm_urdf/piper_x/meshes/dae/flange.dae"/>
+            </geometry>
+        </visual>
+        <collision>
+            <origin xyz="0 0 0" rpy="0 0 0"/>
+            <geometry>
+                <mesh filename="package://agx_arm_description/agx_arm_urdf/piper_x/meshes/flange.stl"/>
+            </geometry>
+        </collision>
+    </link>
+    <joint name="flange_joint" type="fixed">
+        <origin xyz="0 0 0" rpy="0 0 0"/>
+        <parent link="link6"/>
+        <child link="flange_link"/>
+    </joint>
     <link name="gripper_base">
         <inertial>
@@ -24,6 +48,6 @@
     </link>
     <joint name="gripper_base_joint" type="fixed">
-        <origin xyz="0 0 0" rpy="0 0 1.5707963"/>
-        <parent link="link6"/>
+        <origin xyz="0 0 0.0045" rpy="0 0 1.5707963"/>
+        <parent link="flange_link"/>
         <child link="gripper_base"/>
     </joint>
@@ -56,5 +80,5 @@
     </link>
     <joint name="gripper_joint1" type="prismatic">
-        <origin xyz="0 0 0.1358" rpy="1.5707963 0 0"/>
+        <origin xyz="0 0 0.138" rpy="1.5707963 0 0"/>
         <parent link="gripper_base"/>
         <child link="gripper_link1"/>
@@ -83,5 +107,5 @@
     </link>
     <joint name="gripper_joint2" type="prismatic">
-        <origin xyz="0 0 0.1358" rpy="1.5707963 0 -3.1415926"/>
+        <origin xyz="0 0 0.138" rpy="1.5707963 0 -3.1415926"/>
         <parent link="gripper_base"/>
         <child link="gripper_link2"/>

File: piper_x/urdf/piper_x_with_left_revo2_description.xacro (robot description, xacro)
@@ -8,7 +8,7 @@
     <link name="flange_link">
         <inertial>
-            <origin xyz="0.0 0.0 0.004" rpy="0 0 0"/>
-            <mass value="0.001"/>
-            <inertia ixx="0.00000001" ixy="0.00000000" ixz="0.00000000" iyy="0.00000001" iyz="0.00000000" izz="0.00000001"/>
+            <origin xyz="1.151691e-03 0.782428e-03 4.798051e-03" rpy="0 0 0"/>
+            <mass value="0.04"/>
+            <inertia ixx="9.935389e-06" ixy="0.0" ixz="0.0" iyy="10.508003e-06" iyz="0.0" izz="19.652873e-06"/>
         </inertial>
         <visual>
@@ -31,5 +31,5 @@
     </joint>
     <joint name="hand_base_joint" type="fixed">
-        <origin xyz="0.0 0.0 0.008" rpy="0 0 0"/>
+        <origin xyz="0.0 0.0 0.0105" rpy="0 0 0"/>
         <parent link="flange_link"/>
         <child link="left_base_link"/>

File: piper_x/urdf/piper_x_with_right_revo2_description.xacro (robot description, xacro)
@@ -8,7 +8,7 @@
     <link name="flange_link">
         <inertial>
-            <origin xyz="0.0 0.0 0.004" rpy="0 0 0"/>
-            <mass value="0.001"/>
-            <inertia ixx="0.00000001" ixy="0.00000000" ixz="0.00000000" iyy="0.00000001" iyz="0.00000000" izz="0.00000001"/>
+            <origin xyz="1.151691e-03 0.782428e-03 4.798051e-03" rpy="0 0 0"/>
+            <mass value="0.04"/>
+            <inertia ixx="9.935389e-06" ixy="0.0" ixz="0.0" iyy="10.508003e-06" iyz="0.0" izz="19.652873e-06"/>
         </inertial>
         <visual>
@@ -31,5 +31,5 @@
     </joint>
     <joint name="hand_base_joint" type="fixed">
-        <origin xyz="0.0 0.0 0.008" rpy="0 0 0"/>
+        <origin xyz="0.0 0.0 0.0105" rpy="0 0 0"/>
         <parent link="flange_link"/>
         <child link="right_base_link"/>
