Commit message: fix(urdf): Nero Revo2 末端统一使用夹爪法兰
- 左右 Revo2 组合复用 gripper_flange，保持灵巧手安装偏移
- 删除 Revo2 专用法兰 Xacro、STL 和 DAE 模型

---

fix(urdf): use the gripper flange for Nero Revo2 end effectors

- Reuse gripper_flange for both Revo2 hands while preserving hand mounting offsets
- Remove the dedicated Revo2 flange Xacro, STL and DAE models

File: nero/urdf/nero_with_left_revo2_description.xacro (robot description, xacro)
@@ -5,8 +5,8 @@
 <robot xmlns:xacro="http://www.ros.org/wiki/xacro" name="nero">
 <xacro:include filename="$(find agx_arm_description)/agx_arm_urdf/revo2/urdf/revo2_left_hand.urdf"/>
-<xacro:include filename="$(find agx_arm_description)/agx_arm_urdf/nero/urdf/nero_with_revo2_flange_description.xacro"/>
+<xacro:include filename="$(find agx_arm_description)/agx_arm_urdf/nero/urdf/nero_with_gripper_flange_description.xacro"/>
     <joint name="hand_base_joint" type="fixed">
         <origin xyz="0.0 0.0 0.012" rpy="0 0 3.1415926"/>
-        <parent link="revo2_flange"/>
+        <parent link="gripper_flange"/>
         <child link="left_base_link"/>
         <axis xyz="0 0 0"/>

File: nero/urdf/nero_with_right_revo2_description.xacro (robot description, xacro)
@@ -5,8 +5,8 @@
 <robot xmlns:xacro="http://www.ros.org/wiki/xacro" name="nero">
 <xacro:include filename="$(find agx_arm_description)/agx_arm_urdf/revo2/urdf/revo2_right_hand.urdf"/>
-<xacro:include filename="$(find agx_arm_description)/agx_arm_urdf/nero/urdf/nero_with_revo2_flange_description.xacro"/>
+<xacro:include filename="$(find agx_arm_description)/agx_arm_urdf/nero/urdf/nero_with_gripper_flange_description.xacro"/>
     <joint name="hand_base_joint" type="fixed">
         <origin xyz="0.0 0.0 0.012" rpy="0 0 3.1415926"/>
-        <parent link="revo2_flange"/>
+        <parent link="gripper_flange"/>
         <child link="right_base_link"/>
         <axis xyz="0.0 0.0 0.0"/>
