Commit message: fix(urdf): 同步 Nero Revo2 夹爪法兰模型
- 同步 main 提交 c2b15a0，左右 Revo2 末端统一使用 gripper_flange
- 删除 Revo2 专用法兰模型与组合描述，保留当前分支的路径格式和灵巧手安装偏移

---

fix(urdf): sync Nero Revo2 gripper flange models

- Sync main commit c2b15a0 and use gripper_flange for both Revo2 hands
- Remove dedicated Revo2 flange models and descriptions while preserving branch-specific mesh paths and hand mounting offsets

File: nero/urdf/nero_with_left_revo2_description.urdf (robot description, URDF)
Before this commit: robot nero, 32 links, 31 joints
Links:
- removed link revo2_flange
- added link gripper_flange, mass 0.04771096; collision mesh filename=meshes/gripper_flange.stl; visual mesh filename=meshes/dae/gripper_flange.dae
Joints:
- removed joint revo2_flange_joint
- added joint gripper_flange_joint: type fixed, parent link7, child gripper_flange, origin xyz=0.031 0 -0.0235 rpy=-1.5708 0 -1.5708
- joint hand_base_joint: parent revo2_flange -> gripper_flange

File: nero/urdf/nero_with_right_revo2_description.urdf (robot description, URDF)
Before this commit: robot nero, 32 links, 31 joints
Links:
- removed link revo2_flange
- added link gripper_flange, mass 0.04771096; collision mesh filename=meshes/gripper_flange.stl; visual mesh filename=meshes/dae/gripper_flange.dae
Joints:
- removed joint revo2_flange_joint
- added joint gripper_flange_joint: type fixed, parent link7, child gripper_flange, origin xyz=0.031 0 -0.0235 rpy=-1.5708 0 -1.5708
- joint hand_base_joint: parent revo2_flange -> gripper_flange

Commit message: fix(urdf): 同步 Nero Revo2 夹爪法兰模型
- 同步 main 提交 c2b15a0，左右 Revo2 末端统一使用 gripper_flange
- 删除 Revo2 专用法兰模型与组合描述，保留当前分支的路径格式和灵巧手安装偏移

---

fix(urdf): sync Nero Revo2 gripper flange models

- Sync main commit c2b15a0 and use gripper_flange for both Revo2 hands
- Remove dedicated Revo2 flange models and descriptions while preserving branch-specific mesh paths and hand mounting offsets

File: nero/urdf/nero_with_left_revo2_description.urdf (robot description, URDF)
Before this commit: robot nero, 32 links, 31 joints
Links:
- removed link revo2_flange
- added link gripper_flange, mass 0.04771096; collision mesh filename=package://agx_arm_description/agx_arm_urdf/nero/meshes/grip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; visual mesh filename=package://agx_arm_description/agx_arm_urdf/nero/meshes/dae/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
Joints:
- removed joint revo2_flange_joint
- added joint gripper_flange_joint: type fixed, parent link7, child gripper_flange, origin xyz=0.031 0 -0.0235 rpy=-1.5708 0 -1.5708
- joint hand_base_joint: parent revo2_flange -> gripper_flange

File: nero/urdf/nero_with_right_revo2_description.urdf (robot description, URDF)
Before this commit: robot nero, 32 links, 31 joints
Links:
- removed link revo2_flange
- added link gripper_flange, mass 0.04771096; collision mesh filename=package://agx_arm_description/agx_arm_urdf/nero/meshes/grip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; visual mesh filename=package://agx_arm_description/agx_arm_urdf/nero/meshes/dae/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
Joints:
- removed joint revo2_flange_joint
- added joint gripper_flange_joint: type fixed, parent link7, child gripper_flange, origin xyz=0.031 0 -0.0235 rpy=-1.5708 0 -1.5708
- joint hand_base_joint: parent revo2_flange -> gripper_flange
