Commit message: refactor(urdf): 同步共用夹爪与 Nero 法兰命名
- 同步 main 提交 983788b，更新共用夹爪网格并新增独立夹爪 URDF
- Nero 法兰统一为 flange_link/flange_joint，更新夹爪和左右 Revo2 展开模型
- 保留当前分支的网格路径结构；relative 各型号仍可独立使用

- 更新中英文模型列表与目录结构

---

refactor(urdf): sync shared gripper models and Nero flange names

- Sync main commit 983788b: shared gripper meshes and a standalone gripper URDF
- Use flange_link/flange_joint for Nero and update expanded gripper and Revo2 models
- Preserve branch-specific mesh paths and self-contained model directories on relative
- Update bilingual model lists and directory structure

File: nero/urdf/nero_with_flange_description.urdf (robot description, URDF)
Before this commit: robot nero, 14 links, 13 joints
Links:
- removed link gripper_base
- removed link gripper_link
- removed link gripper_link1
- removed link gripper_link2
Joints:
- removed joint gripper
- removed joint gripper_base_joint
- removed joint gripper_joint1
- removed joint gripper_joint2

File: nero/urdf/nero_with_gripper_description.xacro (robot description, xacro)
@@ -3,21 +3,21 @@
      For more information, please see http://wiki.ros.org/sw_urdf_exporter -->
 <robot xmlns:xacro="http://www.ros.org/wiki/xacro" name="nero">
-<xacro:include filename="$(find agx_arm_description)/agx_arm_urdf/nero/urdf/nero_with_gripper_flange_description.xacro"/>
+<xacro:include filename="$(find agx_arm_description)/agx_arm_urdf/nero/urdf/nero_with_flange_description.xacro"/>
     <link name="gripper_base">
         <inertial>
             <origin xyz="-0.000183807162235591 8.05033155577911E-05 0.0321436689908876" rpy="0 0 0"/>
             <mass value="0.45"/>
-            <inertia ixx="0.00092934" ixy="0.00000034" ixz="-0.00000738" iyy="0.00071447" iyz="0.00000005" izz="0.00039442"/>
+            <inertia ixx="0.000466587336445" ixy="0" ixz="0" iyy="0.000208793681739" iyz="0" izz="0.000443633623295"/>
         </inertial>
         <visual>
-            <origin xyz="0 0 0" rpy="0 0 0"/>
+            <origin xyz="0 0 0.000003" rpy="0 0 3.141592653589793"/>
             <geometry>
-                <mesh filename="package://agx_arm_description/agx_arm_urdf/nero/meshes/dae/gripper_base.dae"/>
+                <mesh filename="package://agx_arm_description/agx_arm_urdf/agx_gripper/meshes/dae/gripper_base.dae"/>
             </geometry>
         </visual>
         <collision>
-            <origin xyz="0 0 0" rpy="0 0 0"/>
+            <origin xyz="0 0 0.000003" rpy="0 0 3.141592653589793"/>
             <geometry>
-                <mesh filename="package://agx_arm_description/agx_arm_urdf/nero/meshes/gripper_base.stl"/>
+                <mesh filename="package://agx_arm_description/agx_arm_urdf/agx_gripper/meshes/gripper_base.stl"/>
             </geometry>
         </collision>
@@ -25,5 +25,5 @@
     <joint name="gripper_base_joint" type="fixed">
         <origin xyz="0 0 0.006" rpy="0 0 0"/>
-        <parent link="gripper_flange"/>
+        <parent link="flange_link"/>
         <child link="gripper_base"/>
     </joint>
@@ -40,10 +40,10 @@
             <origin xyz="0.00065123185041968 -0.0491929869131989 0.00972258769184025" rpy="0 0 0"/>
             <mass value="0.025"/>
-            <inertia ixx="0.00007371" ixy="-0.00000113" ixz="0.00000021" iyy="0.00000781" iyz="-0.00001372" izz="0.0000747"/>
+            <inertia ixx="1.0831334372e-05" ixy="3.32108655243e-07" ixz="-5.17776964242e-08" iyy="5.43941050918e-06" iyz="1.75746071559e-06" izz="1.41828415054e-05"/>
         </inertial>
         <visual>
             <origin xyz="0 0 0" rpy="0 0 0"/>
             <geometry>
-                <mesh filename="package://agx_arm_description/agx_arm_urdf/nero/meshes/dae/gripper_link1.dae"/>
+                <mesh filename="package://agx_arm_description/agx_arm_urdf/agx_gripper/meshes/dae/gripper_link1.dae"/>
             </geometry>
         </visual>
@@ -51,5 +51,5 @@
             <origin xyz="0 0 0" rpy="0 0 0"/>
             <geometry>
-                <mesh filename="package://agx_arm_description/agx_arm_urdf/nero/meshes/gripper_link1.stl"/>
+                <mesh filename="package://agx_arm_description/agx_arm_urdf/agx_gripper/meshes/gripper_link1.stl"/>
             </geometry>
         </collision>
@@ -67,10 +67,10 @@
             <origin xyz="0.00065123185041968 -0.0491929869131989 0.00972258769184025" rpy="0 0 0"/>
             <mass value="0.025"/>
-            <inertia ixx="0.00007371" ixy="-0.00000113" ixz="0.00000021" iyy="0.00000781" iyz="-0.00001372" izz="0.0000747"/>
+            <inertia ixx="1.0831334372e-05" ixy="3.32108655243e-07" ixz="-5.17776964242e-08" iyy="5.43941050918e-06" iyz="1.75746071559e-06" izz="1.41828415054e-05"/>
         </inertial>
         <visual>
             <origin xyz="0 0 0" rpy="0 0 0"/>
             <geometry>
-                <mesh filename="package://agx_arm_description/agx_arm_urdf/nero/meshes/dae/gripper_link2.dae"/>
+                <mesh filename="package://agx_arm_description/agx_arm_urdf/agx_gripper/meshes/dae/gripper_link2.dae"/>
             </geometry>
         </visual>
@@ -78,5 +78,5 @@
             <origin xyz="0 0 0" rpy="0 0 0"/>
             <geometry>
-                <mesh filename="package://agx_arm_description/agx_arm_urdf/nero/meshes/gripper_link2.stl"/>
+                <mesh filename="package://agx_arm_description/agx_arm_urdf/agx_gripper/meshes/gripper_link2.stl"/>
             </geometry>
         </collision>

File: nero/urdf/nero_with_left_revo2_description.urdf (robot description, URDF)
Before this commit: robot nero, 32 links, 31 joints
Links:
- removed link gripper_flange
- added link flange_link, mass 0.04771096; collision mesh filename=package://agx_arm_description/agx_arm_urdf/nero/meshes/flan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; visual mesh filename=package://agx_arm_description/agx_arm_urdf/nero/meshes/dae/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
Joints:
- removed joint gripper_flange_joint
- added joint flange_joint: type fixed, parent link7, child flange_link, origin xyz=0.031 0 -0.0235 rpy=-1.5708 0 -1.5708
- joint hand_base_joint: parent gripper_flange -> flange_link

File: nero/urdf/nero_with_right_revo2_description.urdf (robot description, URDF)
Before this commit: robot nero, 32 links, 31 joints
Links:
- removed link gripper_flange
- added link flange_link, mass 0.04771096; collision mesh filename=package://agx_arm_description/agx_arm_urdf/nero/meshes/flan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; visual mesh filename=package://agx_arm_description/agx_arm_urdf/nero/meshes/dae/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
Joints:
- removed joint gripper_flange_joint
- added joint flange_joint: type fixed, parent link7, child flange_link, origin xyz=0.031 0 -0.0235 rpy=-1.5708 0 -1.5708
- joint hand_base_joint: parent gripper_flange -> flange_link

File: piper/urdf/piper_with_gripper_description.urdf (robot description, URDF)
Before this commit: robot piper, 13 links, 12 joints
Links:
- link gripper_base: geometry collision mesh filename=package://agx_arm_description/agx_arm_urdf/agx_gripper/mesh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; visual mesh filename=package://agx_arm_description/agx_arm_urdf/agx_gripper/mesh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
- link gripper_link1: geometry collision mesh filename=package://agx_arm_description/agx_arm_urdf/agx_gripper/mesh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; visual mesh filename=package://agx_arm_description/agx_arm_urdf/agx_gripper/mesh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
- link gripper_link2: geometry collision mesh filename=package://agx_arm_description/agx_arm_urdf/agx_gripper/mesh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; visual mesh filename=package://agx_arm_description/agx_arm_urdf/agx_gripper/mesh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

File: piper_h/urdf/piper_h_with_gripper_description.urdf (robot description, URDF)
Before this commit: robot piper_h, 13 links, 12 joints
Links:
- link gripper_base: geometry collision mesh filename=package://agx_arm_description/agx_arm_urdf/agx_gripper/mesh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; visual mesh filename=package://agx_arm_description/agx_arm_urdf/agx_gripper/mesh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
- link gripper_link1: geometry collision mesh filename=package://agx_arm_description/agx_arm_urdf/agx_gripper/mesh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; visual mesh filename=package://agx_arm_description/agx_arm_urdf/agx_gripper/mesh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
- link gripper_link2: geometry collision mesh filename=package://agx_arm_description/agx_arm_urdf/agx_gripper/mesh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; visual mesh filename=package://agx_arm_description/agx_arm_urdf/agx_gripper/mesh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

File: piper_l/urdf/piper_l_with_gripper_description.urdf (robot description, URDF)
Before this commit: robot piper_l, 13 links, 12 joints
Links:
- link gripper_base: geometry collision mesh filename=package://agx_arm_description/agx_arm_urdf/agx_gripper/mesh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; visual mesh filename=package://agx_arm_description/agx_arm_urdf/agx_gripper/mesh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
- link gripper_link1: geometry collision mesh filename=package://agx_arm_description/agx_arm_urdf/agx_gripper/mesh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; visual mesh filename=package://agx_arm_description/agx_arm_urdf/agx_gripper/mesh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
- link gripper_link2: geometry collision mesh filename=package://agx_arm_description/agx_arm_urdf/agx_gripper/mesh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; visual mesh filename=package://agx_arm_description/agx_arm_urdf/agx_gripper/mesh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

File: piper_x/urdf/piper_x_with_gripper_description.urdf (robot description, URDF)
Before this commit: robot piper_x, 13 links, 12 joints
Links:
- link gripper_base: geometry collision mesh filename=package://agx_arm_description/agx_arm_urdf/agx_gripper/mesh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; visual mesh filename=package://agx_arm_description/agx_arm_urdf/agx_gripper/mesh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
- link gripper_link1: geometry collision mesh filename=package://agx_arm_description/agx_arm_urdf/agx_gripper/mesh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; visual mesh filename=package://agx_arm_description/agx_arm_urdf/agx_gripper/mesh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
- link gripper_link2: geometry collision mesh filename=package://agx_arm_description/agx_arm_urdf/agx_gripper/mesh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; visual mesh filename=package://agx_arm_description/agx_arm_urdf/agx_gripper/mesh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

Commit message: refactor(urdf): 同步共用夹爪与 Nero 法兰命名
- 同步 main 提交 983788b，更新共用夹爪网格并新增独立夹爪 URDF
- Nero 法兰统一为 flange_link/flange_joint，更新夹爪和左右 Revo2 展开模型
- 保留当前分支的网格路径结构；relative 各型号仍可独立使用

- 更新中英文模型列表与目录结构

---

refactor(urdf): sync shared gripper models and Nero flange names

- Sync main commit 983788b: shared gripper meshes and a standalone gripper URDF
- Use flange_link/flange_joint for Nero and update expanded gripper and Revo2 models
- Preserve branch-specific mesh paths and self-contained model directories on relative
- Update bilingual model lists and directory structure

File: nero/urdf/nero_with_flange_description.urdf (robot description, URDF)
Before this commit: robot nero, 14 links, 13 joints
Links:
- removed link gripper_base
- removed link gripper_link
- removed link gripper_link1
- removed link gripper_link2
Joints:
- removed joint gripper
- removed joint gripper_base_joint
- removed joint gripper_joint1
- removed joint gripper_joint2

File: nero/urdf/nero_with_left_revo2_description.urdf (robot description, URDF)
Before this commit: robot nero, 32 links, 31 joints
Links:
- removed link gripper_flange
- added link flange_link, mass 0.04771096; collision mesh filename=meshes/flange.stl; visual mesh filename=meshes/dae/flange.dae
Joints:
- removed joint gripper_flange_joint
- added joint flange_joint: type fixed, parent link7, child flange_link, origin xyz=0.031 0 -0.0235 rpy=-1.5708 0 -1.5708
- joint hand_base_joint: parent gripper_flange -> flange_link

File: nero/urdf/nero_with_right_revo2_description.urdf (robot description, URDF)
Before this commit: robot nero, 32 links, 31 joints
Links:
- removed link gripper_flange
- added link flange_link, mass 0.04771096; collision mesh filename=meshes/flange.stl; visual mesh filename=meshes/dae/flange.dae
Joints:
- removed joint gripper_flange_joint
- added joint flange_joint: type fixed, parent link7, child flange_link, origin xyz=0.031 0 -0.0235 rpy=-1.5708 0 -1.5708
- joint hand_base_joint: parent gripper_flange -> flange_link

File: piper/urdf/piper_with_gripper_description.urdf (robot description, URDF)
Before this commit: robot piper, 13 links, 12 joints
Links:
- link gripper_base: geometry collision mesh filename=meshes/agx_gripper/meshes/gripper_base.stl; visual mesh filename=meshes/agx_gripper/meshes/dae/gripper_base.dae
- link gripper_link1: geometry collision mesh filename=meshes/agx_gripper/meshes/gripper_link1.stl; visual mesh filename=meshes/agx_gripper/meshes/dae/gripper_link1.dae
- link gripper_link2: geometry collision mesh filename=meshes/agx_gripper/meshes/gripper_link2.stl; visual mesh filename=meshes/agx_gripper/meshes/dae/gripper_link2.dae

File: piper_h/urdf/piper_h_with_gripper_description.urdf (robot description, URDF)
Before this commit: robot piper_h, 13 links, 12 joints
Links:
- link gripper_base: geometry collision mesh filename=meshes/agx_gripper/meshes/gripper_base.stl; visual mesh filename=meshes/agx_gripper/meshes/dae/gripper_base.dae
- link gripper_link1: geometry collision mesh filename=meshes/agx_gripper/meshes/gripper_link1.stl; visual mesh filename=meshes/agx_gripper/meshes/dae/gripper_link1.dae
- link gripper_link2: geometry collision mesh filename=meshes/agx_gripper/meshes/gripper_link2.stl; visual mesh filename=meshes/agx_gripper/meshes/dae/gripper_link2.dae

File: piper_l/urdf/piper_l_with_gripper_description.urdf (robot description, URDF)
Before this commit: robot piper_l, 13 links, 12 joints
Links:
- link gripper_base: geometry collision mesh filename=meshes/agx_gripper/meshes/gripper_base.stl; visual mesh filename=meshes/agx_gripper/meshes/dae/gripper_base.dae
- link gripper_link1: geometry collision mesh filename=meshes/agx_gripper/meshes/gripper_link1.stl; visual mesh filename=meshes/agx_gripper/meshes/dae/gripper_link1.dae
- link gripper_link2: geometry collision mesh filename=meshes/agx_gripper/meshes/gripper_link2.stl; visual mesh filename=meshes/agx_gripper/meshes/dae/gripper_link2.dae

File: piper_x/urdf/piper_x_with_gripper_description.urdf (robot description, URDF)
Before this commit: robot piper_x, 13 links, 12 joints
Links:
- link gripper_base: geometry collision mesh filename=meshes/agx_gripper/meshes/gripper_base.stl; visual mesh filename=meshes/agx_gripper/meshes/dae/gripper_base.dae
- link gripper_link1: geometry collision mesh filename=meshes/agx_gripper/meshes/gripper_link1.stl; visual mesh filename=meshes/agx_gripper/meshes/dae/gripper_link1.dae
- link gripper_link2: geometry collision mesh filename=meshes/agx_gripper/meshes/gripper_link2.stl; visual mesh filename=meshes/agx_gripper/meshes/dae/gripper_link2.dae

Commit message: fix(urdf): 同步 Nero 各末端模型 J6 关节限位
将 Nero 基础、法兰、夹爪及左右 Revo2 模型的 J6 限位统一为 -42° 至 50°，保留分支网格路径。

---

fix(urdf): sync Nero J6 limits across end-effector models

Set J6 limits to -42 to 50 degrees for Nero base, flange, gripper and both Revo2 models while preserving branch-specific mesh paths.

File: nero/urdf/nero_with_flange_description.urdf (robot description, URDF)
Before this commit: robot nero, 10 links, 9 joints
Joints:
- joint joint6: limit lower=-0.73 upper=0.95 effort=100 velocity=5 -> lower=-0.7330383 upper=0.8726646 effort=100 velocity=5

File: nero/urdf/nero_with_gripper_description.urdf (robot description, URDF)
Before this commit: robot nero, 14 links, 13 joints
Joints:
- joint joint6: limit lower=-0.73 upper=0.95 effort=100 velocity=5 -> lower=-0.7330383 upper=0.8726646 effort=100 velocity=5

File: nero/urdf/nero_with_left_revo2_description.urdf (robot description, URDF)
Before this commit: robot nero, 32 links, 31 joints
Joints:
- joint joint6: limit lower=-0.73 upper=0.95 effort=100 velocity=5 -> lower=-0.7330383 upper=0.8726646 effort=100 velocity=5

File: nero/urdf/nero_with_right_revo2_description.urdf (robot description, URDF)
Before this commit: robot nero, 32 links, 31 joints
Joints:
- joint joint6: limit lower=-0.73 upper=0.95 effort=100 velocity=5 -> lower=-0.7330383 upper=0.8726646 effort=100 velocity=5
