Commit message: refactor(urdf): 共用夹爪网格并统一 Nero 法兰命名
- 将夹爪基座和两片夹片网格集中到 agx_gripper，新增独立夹爪 URDF，减少重复文件
- Nero 复用 Piper 基座网格，通过 visual/collision 原点补偿保持安装方向和关节运动不变
- 将 Nero 法兰统一为 flange_link、flange_joint、flange 网格及描述文件，并同步 Revo2 引用

- 更新中英文模型列表与目录结构

---

refactor(urdf): share gripper meshes and unify Nero flange names

- Consolidate gripper base and finger meshes under agx_gripper and add a standalone gripper URDF
- Reuse Piper base meshes for Nero with visual/collision origin compensation, preserving mounting orientation and joint motion
- Rename the Nero flange to flange_link/flange_joint, update flange mesh and description filenames, and synchronize Revo2 references
- Update bilingual model lists and directory structure

File: agx_gripper/urdf/agx_gripper_description.urdf (robot description, URDF)
Before this commit: robot nero, 4 links, 4 joints
Joints:
- removed joint gripper_base_joint
- joint gripper_joint1: origin xyz=0 0 0.138 rpy=1.5707963 0 3.1415926 -> xyz=0 0 0.138 rpy=1.5707963 0 0
- joint gripper_joint2: origin xyz=0 0 0.138 rpy=1.5707963 0 0 -> xyz=0 0 0.138 rpy=1.5707963 0 -3.1415926

File: nero/urdf/nero_with_flange_description.xacro (robot description, xacro)
@@ -4,5 +4,5 @@
 <robot xmlns:xacro="http://www.ros.org/wiki/xacro" name="nero">
 <xacro:include filename="$(find agx_arm_description)/agx_arm_urdf/nero/urdf/nero_description.urdf"/>
-    <link name="gripper_flange">
+    <link name="flange_link">
         <inertial>
             <origin xyz="0.000253201 -0.000322696 -0.010082901" rpy="0 0 0"/>
@@ -13,5 +13,5 @@
             <origin xyz="0 0 0" rpy="0 0 0"/>
             <geometry>
-                <mesh filename="package://agx_arm_description/agx_arm_urdf/nero/meshes/dae/gripper_flange.dae"/>
+                <mesh filename="package://agx_arm_description/agx_arm_urdf/nero/meshes/dae/flange.dae"/>
             </geometry>
         </visual>
@@ -19,12 +19,12 @@
             <origin xyz="0 0 0" rpy="0 0 0"/>
             <geometry>
-                <mesh filename="package://agx_arm_description/agx_arm_urdf/nero/meshes/gripper_flange.stl"/>
+                <mesh filename="package://agx_arm_description/agx_arm_urdf/nero/meshes/flange.stl"/>
             </geometry>
         </collision>
     </link>
-    <joint name="gripper_flange_joint" type="fixed">
+    <joint name="flange_joint" type="fixed">
         <origin xyz="0.031 0 -0.0235" rpy="-1.5708 0 -1.5708"/>
         <parent link="link7"/>
-        <child link="gripper_flange"/>
+        <child link="flange_link"/>
     </joint>
 </robot>

File: nero/urdf/nero_with_left_revo2_description.xacro (robot description, xacro)
@@ -5,8 +5,8 @@
 <robot xmlns:xacro="http://www.ros.org/wiki/xacro" name="nero">
 <xacro:include filename="$(find agx_arm_description)/agx_arm_urdf/revo2/urdf/revo2_left_hand.urdf"/>
-<xacro:include filename="$(find agx_arm_description)/agx_arm_urdf/nero/urdf/nero_with_gripper_flange_description.xacro"/>
+<xacro:include filename="$(find agx_arm_description)/agx_arm_urdf/nero/urdf/nero_with_flange_description.xacro"/>
     <joint name="hand_base_joint" type="fixed">
         <origin xyz="0.0 0.0 0.012" rpy="0 0 3.1415926"/>
-        <parent link="gripper_flange"/>
+        <parent link="flange_link"/>
         <child link="left_base_link"/>
         <axis xyz="0 0 0"/>

File: nero/urdf/nero_with_right_revo2_description.xacro (robot description, xacro)
@@ -5,8 +5,8 @@
 <robot xmlns:xacro="http://www.ros.org/wiki/xacro" name="nero">
 <xacro:include filename="$(find agx_arm_description)/agx_arm_urdf/revo2/urdf/revo2_right_hand.urdf"/>
-<xacro:include filename="$(find agx_arm_description)/agx_arm_urdf/nero/urdf/nero_with_gripper_flange_description.xacro"/>
+<xacro:include filename="$(find agx_arm_description)/agx_arm_urdf/nero/urdf/nero_with_flange_description.xacro"/>
     <joint name="hand_base_joint" type="fixed">
         <origin xyz="0.0 0.0 0.012" rpy="0 0 3.1415926"/>
-        <parent link="gripper_flange"/>
+        <parent link="flange_link"/>
         <child link="right_base_link"/>
         <axis xyz="0.0 0.0 0.0"/>

File: piper/urdf/piper_with_gripper_description.xacro (robot description, xacro)
@@ -32,10 +32,10 @@
             <origin xyz="-0.000183807162235591 8.05033155577911E-05 0.0321436689908876" rpy="0 0 0"/>
             <mass value="0.45"/>
-            <inertia ixx="0.00092934" ixy="0.00000034" ixz="-0.00000738" iyy="0.00071447" iyz="0.00000005" izz="0.00039442"/>
+            <inertia ixx="0.000466573035886" ixy="0" ixz="0" iyy="0.000208671755285" iyz="0" izz="0.000443517627645"/>
         </inertial>
         <visual>
             <origin xyz="0 0 0" rpy="0 0 0"/>
             <geometry>
-                <mesh filename="package://agx_arm_description/agx_arm_urdf/piper/meshes/dae/gripper_base.dae"/>
+                <mesh filename="package://agx_arm_description/agx_arm_urdf/agx_gripper/meshes/dae/gripper_base.dae"/>
             </geometry>
         </visual>
@@ -43,5 +43,5 @@
             <origin xyz="0 0 0" rpy="0 0 0"/>
             <geometry>
-                <mesh filename="package://agx_arm_description/agx_arm_urdf/piper/meshes/gripper_base.stl"/>
+                <mesh filename="package://agx_arm_description/agx_arm_urdf/agx_gripper/meshes/gripper_base.stl"/>
             </geometry>
         </collision>
@@ -64,10 +64,10 @@
             <origin xyz="0.00065123185041968 -0.0491929869131989 0.00972258769184025" rpy="0 0 0"/>
             <mass value="0.025"/>
-            <inertia ixx="0.00007371" ixy="-0.00000113" ixz="0.00000021" iyy="0.00000781" iyz="-0.00001372" izz="0.0000747"/>
+            <inertia ixx="1.0831334372e-05" ixy="3.32108655243e-07" ixz="-5.17776964242e-08" iyy="5.43941050918e-06" iyz="1.75746071559e-06" izz="1.41828415054e-05"/>
         </inertial>
         <visual>
             <origin xyz="0 0 0" rpy="0 0 0"/>
             <geometry>
-                <mesh filename="package://agx_arm_description/agx_arm_urdf/piper/meshes/dae/gripper_link1.dae"/>
+                <mesh filename="package://agx_arm_description/agx_arm_urdf/agx_gripper/meshes/dae/gripper_link1.dae"/>
             </geometry>
         </visual>
@@ -75,5 +75,5 @@
             <origin xyz="0 0 0" rpy="0 0 0"/>
             <geometry>
-                <mesh filename="package://agx_arm_description/agx_arm_urdf/piper/meshes/gripper_link1.stl"/>
+                <mesh filename="package://agx_arm_description/agx_arm_urdf/agx_gripper/meshes/gripper_link1.stl"/>
             </geometry>
         </collision>
@@ -91,10 +91,10 @@
             <origin xyz="0.00065123185041968 -0.0491929869131989 0.00972258769184025" rpy="0 0 0"/>
             <mass value="0.025"/>
-            <inertia ixx="0.00007371" ixy="-0.00000113" ixz="0.00000021" iyy="0.00000781" iyz="-0.00001372" izz="0.0000747"/>
+            <inertia ixx="1.0831334372e-05" ixy="3.32108655243e-07" ixz="-5.17776964242e-08" iyy="5.43941050918e-06" iyz="1.75746071559e-06" izz="1.41828415054e-05"/>
         </inertial>
         <visual>
             <origin xyz="0 0 0" rpy="0 0 0"/>
             <geometry>
-                <mesh filename="package://agx_arm_description/agx_arm_urdf/piper/meshes/dae/gripper_link2.dae"/>
+                <mesh filename="package://agx_arm_description/agx_arm_urdf/agx_gripper/meshes/dae/gripper_link2.dae"/>
             </geometry>
         </visual>
@@ -102,5 +102,5 @@
             <origin xyz="0 0 0" rpy="0 0 0"/>
             <geometry>
-                <mesh filename="package://agx_arm_description/agx_arm_urdf/piper/meshes/gripper_link2.stl"/>
+                <mesh filename="package://agx_arm_description/agx_arm_urdf/agx_gripper/meshes/gripper_link2.stl"/>
             </geometry>
         </collision>

File: piper_h/urdf/piper_h_with_gripper_description.xacro (robot description, xacro)
@@ -32,10 +32,10 @@
             <origin xyz="-0.000183807162235591 8.05033155577911E-05 0.0321436689908876" rpy="0 0 0"/>
             <mass value="0.45"/>
-            <inertia ixx="0.00092934" ixy="0.00000034" ixz="-0.00000738" iyy="0.00071447" iyz="0.00000005" izz="0.00039442"/>
+            <inertia ixx="0.000466573035886" ixy="0" ixz="0" iyy="0.000208671755285" iyz="0" izz="0.000443517627645"/>
         </inertial>
         <visual>
             <origin xyz="0 0 0" rpy="0 0 0"/>
             <geometry>
-                <mesh filename="package://agx_arm_description/agx_arm_urdf/piper_h/meshes/dae/gripper_base.dae"/>
+                <mesh filename="package://agx_arm_description/agx_arm_urdf/agx_gripper/meshes/dae/gripper_base.dae"/>
             </geometry>
         </visual>
@@ -43,5 +43,5 @@
             <origin xyz="0 0 0" rpy="0 0 0"/>
             <geometry>
-                <mesh filename="package://agx_arm_description/agx_arm_urdf/piper_h/meshes/gripper_base.stl"/>
+                <mesh filename="package://agx_arm_description/agx_arm_urdf/agx_gripper/meshes/gripper_base.stl"/>
             </geometry>
         </collision>
@@ -64,10 +64,10 @@
             <origin xyz="0.00065123185041968 -0.0491929869131989 0.00972258769184025" rpy="0 0 0"/>
             <mass value="0.025"/>
-            <inertia ixx="0.00007371" ixy="-0.00000113" ixz="0.00000021" iyy="0.00000781" iyz="-0.00001372" izz="0.0000747"/>
+            <inertia ixx="1.0831334372e-05" ixy="3.32108655243e-07" ixz="-5.17776964242e-08" iyy="5.43941050918e-06" iyz="1.75746071559e-06" izz="1.41828415054e-05"/>
         </inertial>
         <visual>
             <origin xyz="0 0 0" rpy="0 0 0"/>
             <geometry>
-                <mesh filename="package://agx_arm_description/agx_arm_urdf/piper_h/meshes/dae/gripper_link1.dae"/>
+                <mesh filename="package://agx_arm_description/agx_arm_urdf/agx_gripper/meshes/dae/gripper_link1.dae"/>
             </geometry>
         </visual>
@@ -75,5 +75,5 @@
             <origin xyz="0 0 0" rpy="0 0 0"/>
             <geometry>
-                <mesh filename="package://agx_arm_description/agx_arm_urdf/piper_h/meshes/gripper_link1.stl"/>
+                <mesh filename="package://agx_arm_description/agx_arm_urdf/agx_gripper/meshes/gripper_link1.stl"/>
             </geometry>
         </collision>
@@ -91,10 +91,10 @@
             <origin xyz="0.00065123185041968 -0.0491929869131989 0.00972258769184025" rpy="0 0 0"/>
             <mass value="0.025"/>
-            <inertia ixx="0.00007371" ixy="-0.00000113" ixz="0.00000021" iyy="0.00000781" iyz="-0.00001372" izz="0.0000747"/>
+            <inertia ixx="1.0831334372e-05" ixy="3.32108655243e-07" ixz="-5.17776964242e-08" iyy="5.43941050918e-06" iyz="1.75746071559e-06" izz="1.41828415054e-05"/>
         </inertial>
         <visual>
             <origin xyz="0 0 0" rpy="0 0 0"/>
             <geometry>
-                <mesh filename="package://agx_arm_description/agx_arm_urdf/piper_h/meshes/dae/gripper_link2.dae"/>
+                <mesh filename="package://agx_arm_description/agx_arm_urdf/agx_gripper/meshes/dae/gripper_link2.dae"/>
             </geometry>
         </visual>
@@ -102,5 +102,5 @@
             <origin xyz="0 0 0" rpy="0 0 0"/>
             <geometry>
-                <mesh filename="package://agx_arm_description/agx_arm_urdf/piper_h/meshes/gripper_link2.stl"/>
+                <mesh filename="package://agx_arm_description/agx_arm_urdf/agx_gripper/meshes/gripper_link2.stl"/>
             </geometry>
         </collision>

File: piper_l/urdf/piper_l_with_gripper_description.xacro (robot description, xacro)
@@ -32,10 +32,10 @@
             <origin xyz="-0.000183807162235591 8.05033155577911E-05 0.0321436689908876" rpy="0 0 0"/>
             <mass value="0.45"/>
-            <inertia ixx="0.00092934" ixy="0.00000034" ixz="-0.00000738" iyy="0.00071447" iyz="0.00000005" izz="0.00039442"/>
+            <inertia ixx="0.000466573035886" ixy="0" ixz="0" iyy="0.000208671755285" iyz="0" izz="0.000443517627645"/>
         </inertial>
         <visual>
             <origin xyz="0 0 0" rpy="0 0 0"/>
             <geometry>
-                <mesh filename="package://agx_arm_description/agx_arm_urdf/piper_l/meshes/dae/gripper_base.dae"/>
+                <mesh filename="package://agx_arm_description/agx_arm_urdf/agx_gripper/meshes/dae/gripper_base.dae"/>
             </geometry>
         </visual>
@@ -43,5 +43,5 @@
             <origin xyz="0 0 0" rpy="0 0 0"/>
             <geometry>
-                <mesh filename="package://agx_arm_description/agx_arm_urdf/piper_l/meshes/gripper_base.stl"/>
+                <mesh filename="package://agx_arm_description/agx_arm_urdf/agx_gripper/meshes/gripper_base.stl"/>
             </geometry>
         </collision>
@@ -64,10 +64,10 @@
             <origin xyz="0.00065123185041968 -0.0491929869131989 0.00972258769184025" rpy="0 0 0"/>
             <mass value="0.025"/>
-            <inertia ixx="0.00007371" ixy="-0.00000113" ixz="0.00000021" iyy="0.00000781" iyz="-0.00001372" izz="0.0000747"/>
+            <inertia ixx="1.0831334372e-05" ixy="3.32108655243e-07" ixz="-5.17776964242e-08" iyy="5.43941050918e-06" iyz="1.75746071559e-06" izz="1.41828415054e-05"/>
         </inertial>
         <visual>
             <origin xyz="0 0 0" rpy="0 0 0"/>
             <geometry>
-                <mesh filename="package://agx_arm_description/agx_arm_urdf/piper_l/meshes/dae/gripper_link1.dae"/>
+                <mesh filename="package://agx_arm_description/agx_arm_urdf/agx_gripper/meshes/dae/gripper_link1.dae"/>
             </geometry>
         </visual>
@@ -75,5 +75,5 @@
             <origin xyz="0 0 0" rpy="0 0 0"/>
             <geometry>
-                <mesh filename="package://agx_arm_description/agx_arm_urdf/piper_l/meshes/gripper_link1.stl"/>
+                <mesh filename="package://agx_arm_description/agx_arm_urdf/agx_gripper/meshes/gripper_link1.stl"/>
             </geometry>
         </collision>
@@ -91,10 +91,10 @@
             <origin xyz="0.00065123185041968 -0.0491929869131989 0.00972258769184025" rpy="0 0 0"/>
             <mass value="0.025"/>
-            <inertia ixx="0.00007371" ixy="-0.00000113" ixz="0.00000021" iyy="0.00000781" iyz="-0.00001372" izz="0.0000747"/>
+            <inertia ixx="1.0831334372e-05" ixy="3.32108655243e-07" ixz="-5.17776964242e-08" iyy="5.43941050918e-06" iyz="1.75746071559e-06" izz="1.41828415054e-05"/>
         </inertial>
         <visual>
             <origin xyz="0 0 0" rpy="0 0 0"/>
             <geometry>
-                <mesh filename="package://agx_arm_description/agx_arm_urdf/piper_l/meshes/dae/gripper_link2.dae"/>
+                <mesh filename="package://agx_arm_description/agx_arm_urdf/agx_gripper/meshes/dae/gripper_link2.dae"/>
             </geometry>
         </visual>
@@ -102,5 +102,5 @@
             <origin xyz="0 0 0" rpy="0 0 0"/>
             <geometry>
-                <mesh filename="package://agx_arm_description/agx_arm_urdf/piper_l/meshes/gripper_link2.stl"/>
+                <mesh filename="package://agx_arm_description/agx_arm_urdf/agx_gripper/meshes/gripper_link2.stl"/>
             </geometry>
         </collision>

File: piper_x/urdf/piper_x_with_gripper_description.xacro (robot description, xacro)
@@ -32,10 +32,10 @@
             <origin xyz="-0.000183807162235591 8.05033155577911E-05 0.0321436689908876" rpy="0 0 0"/>
             <mass value="0.45"/>
-            <inertia ixx="0.00092934" ixy="0.00000034" ixz="-0.00000738" iyy="0.00071447" iyz="0.00000005" izz="0.00039442"/>
+            <inertia ixx="0.000466573035886" ixy="0" ixz="0" iyy="0.000208671755285" iyz="0" izz="0.000443517627645"/>
         </inertial>
         <visual>
             <origin xyz="0 0 0" rpy="0 0 0"/>
             <geometry>
-                <mesh filename="package://agx_arm_description/agx_arm_urdf/piper_x/meshes/dae/gripper_base.dae"/>
+                <mesh filename="package://agx_arm_description/agx_arm_urdf/agx_gripper/meshes/dae/gripper_base.dae"/>
             </geometry>
         </visual>
@@ -43,5 +43,5 @@
             <origin xyz="0 0 0" rpy="0 0 0"/>
             <geometry>
-                <mesh filename="package://agx_arm_description/agx_arm_urdf/piper_x/meshes/gripper_base.stl"/>
+                <mesh filename="package://agx_arm_description/agx_arm_urdf/agx_gripper/meshes/gripper_base.stl"/>
             </geometry>
         </collision>
@@ -64,10 +64,10 @@
             <origin xyz="0.00065123185041968 -0.0491929869131989 0.00972258769184025" rpy="0 0 0"/>
             <mass value="0.025"/>
-            <inertia ixx="0.00007371" ixy="-0.00000113" ixz="0.00000021" iyy="0.00000781" iyz="-0.00001372" izz="0.0000747"/>
+            <inertia ixx="1.0831334372e-05" ixy="3.32108655243e-07" ixz="-5.17776964242e-08" iyy="5.43941050918e-06" iyz="1.75746071559e-06" izz="1.41828415054e-05"/>
         </inertial>
         <visual>
             <origin xyz="0 0 0" rpy="0 0 0"/>
             <geometry>
-                <mesh filename="package://agx_arm_description/agx_arm_urdf/piper_x/meshes/dae/gripper_link1.dae"/>
+                <mesh filename="package://agx_arm_description/agx_arm_urdf/agx_gripper/meshes/dae/gripper_link1.dae"/>
             </geometry>
         </visual>
@@ -75,5 +75,5 @@
             <origin xyz="0 0 0" rpy="0 0 0"/>
             <geometry>
-                <mesh filename="package://agx_arm_description/agx_arm_urdf/piper_x/meshes/gripper_link1.stl"/>
+                <mesh filename="package://agx_arm_description/agx_arm_urdf/agx_gripper/meshes/gripper_link1.stl"/>
             </geometry>
         </collision>
@@ -91,10 +91,10 @@
             <origin xyz="0.00065123185041968 -0.0491929869131989 0.00972258769184025" rpy="0 0 0"/>
             <mass value="0.025"/>
-            <inertia ixx="0.00007371" ixy="-0.00000113" ixz="0.00000021" iyy="0.00000781" iyz="-0.00001372" izz="0.0000747"/>
+            <inertia ixx="1.0831334372e-05" ixy="3.32108655243e-07" ixz="-5.17776964242e-08" iyy="5.43941050918e-06" iyz="1.75746071559e-06" izz="1.41828415054e-05"/>
         </inertial>
         <visual>
             <origin xyz="0 0 0" rpy="0 0 0"/>
             <geometry>
-                <mesh filename="package://agx_arm_description/agx_arm_urdf/piper_x/meshes/dae/gripper_link2.dae"/>
+                <mesh filename="package://agx_arm_description/agx_arm_urdf/agx_gripper/meshes/dae/gripper_link2.dae"/>
             </geometry>
         </visual>
@@ -102,5 +102,5 @@
             <origin xyz="0 0 0" rpy="0 0 0"/>
             <geometry>
-                <mesh filename="package://agx_arm_description/agx_arm_urdf/piper_x/meshes/gripper_link2.stl"/>
+                <mesh filename="package://agx_arm_description/agx_arm_urdf/agx_gripper/meshes/gripper_link2.stl"/>
             </geometry>
         </collision>
