Commit message: fix(urdf): 修正 Piper 各型号 J6 关节限位
- 将 Piper、Piper H/L/X 的 J6 位置限位由 ±120° 更新为 ±170°
- 保持其余关节限位、力矩和速度参数不变

---

fix(urdf): correct J6 joint limits across Piper variants

- Update J6 position limits from ±120° to ±170° for Piper and Piper H/L/X
- Keep other joint limits, effort and velocity parameters unchanged

File: piper/urdf/piper_description.urdf (robot description, URDF)
Before this commit: robot piper, 8 links, 7 joints
Joints:
- joint joint6: limit lower=-2.0943951 upper=2.0943951 effort=100 velocity=5 -> lower=-2.9670597 upper=2.9670597 effort=100 velocity=5

File: piper_h/urdf/piper_h_description.urdf (robot description, URDF)
Before this commit: robot piper_h, 8 links, 7 joints
Joints:
- joint joint6: limit lower=-2.0943951 upper=2.0943951 effort=100 velocity=5 -> lower=-2.9670597 upper=2.9670597 effort=100 velocity=5

File: piper_l/urdf/piper_l_description.urdf (robot description, URDF)
Before this commit: robot piper_l, 8 links, 7 joints
Joints:
- joint joint6: limit lower=-2.0943951 upper=2.0943951 effort=100 velocity=5 -> lower=-2.9670597 upper=2.9670597 effort=100 velocity=5

File: piper_x/urdf/piper_x_description.urdf (robot description, URDF)
Before this commit: robot piper_x, 8 links, 7 joints
Joints:
- joint joint6: limit lower=-2.0943951 upper=2.0943951 effort=100 velocity=5 -> lower=-2.9670597 upper=2.9670597 effort=100 velocity=5

Commit message: fix(urdf): 同步 Piper 各型号及末端模型 J6 关节限位
- 将 Piper、Piper H/L/X 的基础模型及夹爪、左右 Revo2 模型 J6 限位统一为 ±170°
- 保持各分支资源路径、其余关节限位、力矩和速度参数不变

---

fix(urdf): sync J6 joint limits for Piper variants and end-effector models

- Set J6 limits to ±170° in base, gripper and left/right Revo2 models for Piper and Piper H/L/X
- Preserve branch-specific resource paths, other joint limits, effort and velocity parameters

File: piper/urdf/piper_description.urdf (robot description, URDF)
Before this commit: robot piper, 8 links, 7 joints
Joints:
- joint joint6: limit lower=-2.0943951 upper=2.0943951 effort=100 velocity=5 -> lower=-2.9670597 upper=2.9670597 effort=100 velocity=5

File: piper/urdf/piper_with_gripper_description.urdf (robot description, URDF)
Before this commit: robot piper, 13 links, 12 joints
Joints:
- joint joint6: limit lower=-2.0943951 upper=2.0943951 effort=100 velocity=5 -> lower=-2.9670597 upper=2.9670597 effort=100 velocity=5

File: piper/urdf/piper_with_left_revo2_description.urdf (robot description, URDF)
Before this commit: robot piper, 31 links, 30 joints
Joints:
- joint joint6: limit lower=-2.0943951 upper=2.0943951 effort=100 velocity=5 -> lower=-2.9670597 upper=2.9670597 effort=100 velocity=5

File: piper/urdf/piper_with_right_revo2_description.urdf (robot description, URDF)
Before this commit: robot piper, 31 links, 30 joints
Joints:
- joint joint6: limit lower=-2.0943951 upper=2.0943951 effort=100 velocity=5 -> lower=-2.9670597 upper=2.9670597 effort=100 velocity=5

File: piper_h/urdf/piper_h_description.urdf (robot description, URDF)
Before this commit: robot piper_h, 8 links, 7 joints
Joints:
- joint joint6: limit lower=-2.0943951 upper=2.0943951 effort=100 velocity=5 -> lower=-2.9670597 upper=2.9670597 effort=100 velocity=5

File: piper_h/urdf/piper_h_with_gripper_description.urdf (robot description, URDF)
Before this commit: robot piper_h, 13 links, 12 joints
Joints:
- joint joint6: limit lower=-2.0943951 upper=2.0943951 effort=100 velocity=5 -> lower=-2.9670597 upper=2.9670597 effort=100 velocity=5

File: piper_h/urdf/piper_h_with_left_revo2_description.urdf (robot description, URDF)
Before this commit: robot piper_h, 31 links, 30 joints
Joints:
- joint joint6: limit lower=-2.0943951 upper=2.0943951 effort=100 velocity=5 -> lower=-2.9670597 upper=2.9670597 effort=100 velocity=5

File: piper_h/urdf/piper_h_with_right_revo2_description.urdf (robot description, URDF)
Before this commit: robot piper_h, 31 links, 30 joints
Joints:
- joint joint6: limit lower=-2.0943951 upper=2.0943951 effort=100 velocity=5 -> lower=-2.9670597 upper=2.9670597 effort=100 velocity=5

File: piper_l/urdf/piper_l_description.urdf (robot description, URDF)
Before this commit: robot piper_l, 8 links, 7 joints
Joints:
- joint joint6: limit lower=-2.0943951 upper=2.0943951 effort=100 velocity=5 -> lower=-2.9670597 upper=2.9670597 effort=100 velocity=5

File: piper_l/urdf/piper_l_with_gripper_description.urdf (robot description, URDF)
Before this commit: robot piper_l, 13 links, 12 joints
Joints:
- joint joint6: limit lower=-2.0943951 upper=2.0943951 effort=100 velocity=5 -> lower=-2.9670597 upper=2.9670597 effort=100 velocity=5

File: piper_l/urdf/piper_l_with_left_revo2_description.urdf (robot description, URDF)
Before this commit: robot piper_l, 31 links, 30 joints
Joints:
- joint joint6: limit lower=-2.0943951 upper=2.0943951 effort=100 velocity=5 -> lower=-2.9670597 upper=2.9670597 effort=100 velocity=5

File: piper_l/urdf/piper_l_with_right_revo2_description.urdf (robot description, URDF)
Before this commit: robot piper_l, 31 links, 30 joints
Joints:
- joint joint6: limit lower=-2.0943951 upper=2.0943951 effort=100 velocity=5 -> lower=-2.9670597 upper=2.9670597 effort=100 velocity=5

File: piper_x/urdf/piper_x_description.urdf (robot description, URDF)
Before this commit: robot piper_x, 8 links, 7 joints
Joints:
- joint joint6: limit lower=-2.0943951 upper=2.0943951 effort=100 velocity=5 -> lower=-2.9670597 upper=2.9670597 effort=100 velocity=5

File: piper_x/urdf/piper_x_with_gripper_description.urdf (robot description, URDF)
Before this commit: robot piper_x, 13 links, 12 joints
Joints:
- joint joint6: limit lower=-2.0943951 upper=2.0943951 effort=100 velocity=5 -> lower=-2.9670597 upper=2.9670597 effort=100 velocity=5

File: piper_x/urdf/piper_x_with_left_revo2_description.urdf (robot description, URDF)
Before this commit: robot piper_x, 31 links, 30 joints
Joints:
- joint joint6: limit lower=-2.0943951 upper=2.0943951 effort=100 velocity=5 -> lower=-2.9670597 upper=2.9670597 effort=100 velocity=5

File: piper_x/urdf/piper_x_with_right_revo2_description.urdf (robot description, URDF)
Before this commit: robot piper_x, 31 links, 30 joints
Joints:
- joint joint6: limit lower=-2.0943951 upper=2.0943951 effort=100 velocity=5 -> lower=-2.9670597 upper=2.9670597 effort=100 velocity=5

Commit message: fix(urdf): 修正 Piper 全系列 link6 惯性参数
依据 CAD 质量属性统一更新 Piper、Piper H、Piper L、Piper X 的 link6 质量、质心及惯性张量。

---

fix(urdf): correct link6 inertial parameters for all Piper models

Update link6 mass, center of mass, and inertia tensor for Piper, Piper H, Piper L, and Piper X using CAD mass properties.

File: piper/urdf/piper_description.urdf (robot description, URDF)
Before this commit: robot piper, 8 links, 7 joints
Links:
- link link6: mass 0.00613114124 -> 0.01655408133

File: piper_h/urdf/piper_h_description.urdf (robot description, URDF)
Before this commit: robot piper_h, 8 links, 7 joints
Links:
- link link6: mass 0.00613114124 -> 0.01655408133

File: piper_l/urdf/piper_l_description.urdf (robot description, URDF)
Before this commit: robot piper_l, 8 links, 7 joints
Links:
- link link6: mass 0.00613114124 -> 0.01655408133

File: piper_x/urdf/piper_x_description.urdf (robot description, URDF)
Before this commit: robot piper_x, 8 links, 7 joints
Links:
- link link6: mass 0.00613114124 -> 0.01655408133

Commit message: fix(urdf): 同步 Piper 全系列各末端模型 link6 惯性参数
依据 CAD 质量属性更新四个型号的基础、夹爪和左右 Revo2 模型，保留分支网格路径及其他参数。

---

fix(urdf): sync link6 inertial parameters across all Piper end-effector models

Update base, gripper, and left/right Revo2 models for all four Piper variants using CAD mass properties, preserving branch-specific mesh paths and other parameters.

File: piper/urdf/piper_description.urdf (robot description, URDF)
Before this commit: robot piper, 8 links, 7 joints
Links:
- link link6: mass 0.00613114124 -> 0.01655408133

File: piper/urdf/piper_with_gripper_description.urdf (robot description, URDF)
Before this commit: robot piper, 13 links, 12 joints
Links:
- link link6: mass 0.00613114124 -> 0.01655408133

File: piper/urdf/piper_with_left_revo2_description.urdf (robot description, URDF)
Before this commit: robot piper, 31 links, 30 joints
Links:
- link link6: mass 0.00613114124 -> 0.01655408133

File: piper/urdf/piper_with_right_revo2_description.urdf (robot description, URDF)
Before this commit: robot piper, 31 links, 30 joints
Links:
- link link6: mass 0.00613114124 -> 0.01655408133

File: piper_h/urdf/piper_h_description.urdf (robot description, URDF)
Before this commit: robot piper_h, 8 links, 7 joints
Links:
- link link6: mass 0.00613114124 -> 0.01655408133

File: piper_h/urdf/piper_h_with_gripper_description.urdf (robot description, URDF)
Before this commit: robot piper_h, 13 links, 12 joints
Links:
- link link6: mass 0.00613114124 -> 0.01655408133

File: piper_h/urdf/piper_h_with_left_revo2_description.urdf (robot description, URDF)
Before this commit: robot piper_h, 31 links, 30 joints
Links:
- link link6: mass 0.00613114124 -> 0.01655408133

File: piper_h/urdf/piper_h_with_right_revo2_description.urdf (robot description, URDF)
Before this commit: robot piper_h, 31 links, 30 joints
Links:
- link link6: mass 0.00613114124 -> 0.01655408133

File: piper_l/urdf/piper_l_description.urdf (robot description, URDF)
Before this commit: robot piper_l, 8 links, 7 joints
Links:
- link link6: mass 0.00613114124 -> 0.01655408133

File: piper_l/urdf/piper_l_with_gripper_description.urdf (robot description, URDF)
Before this commit: robot piper_l, 13 links, 12 joints
Links:
- link link6: mass 0.00613114124 -> 0.01655408133

File: piper_l/urdf/piper_l_with_left_revo2_description.urdf (robot description, URDF)
Before this commit: robot piper_l, 31 links, 30 joints
Links:
- link link6: mass 0.00613114124 -> 0.01655408133

File: piper_l/urdf/piper_l_with_right_revo2_description.urdf (robot description, URDF)
Before this commit: robot piper_l, 31 links, 30 joints
Links:
- link link6: mass 0.00613114124 -> 0.01655408133

File: piper_x/urdf/piper_x_description.urdf (robot description, URDF)
Before this commit: robot piper_x, 8 links, 7 joints
Links:
- link link6: mass 0.00613114124 -> 0.01655408133

File: piper_x/urdf/piper_x_with_gripper_description.urdf (robot description, URDF)
Before this commit: robot piper_x, 13 links, 12 joints
Links:
- link link6: mass 0.00613114124 -> 0.01655408133

File: piper_x/urdf/piper_x_with_left_revo2_description.urdf (robot description, URDF)
Before this commit: robot piper_x, 31 links, 30 joints
Links:
- link link6: mass 0.00613114124 -> 0.01655408133

File: piper_x/urdf/piper_x_with_right_revo2_description.urdf (robot description, URDF)
Before this commit: robot piper_x, 31 links, 30 joints
Links:
- link link6: mass 0.00613114124 -> 0.01655408133
